File: hardware/mcu.kicad_sch (KiCad schematic)
At the start: 32 parts, among them J201 2x5 1.27mm, J202 USB_C_Receptacle_USB2.0, U104 RP2040, U202 USBLC6-2SC6, Y201 Crystal_GND24

Commit message: Finished mcu schematic with the rp2040
Parts:
- added C217: 1u, Capacitor_SMD:C_0402_1005Metric, symbol Device:C
- added C218: 100n, Capacitor_SMD:C_0402_1005Metric, symbol Device:C
- added D301: Act, LED_SMD:LED_0603_1608Metric, symbol Device:LED_Filled
- added R201, R202: 27, Resistor_SMD:R_0402_1005Metric, symbol Device:R
- added R212: 10k, Resistor_SMD:R_0402_1005Metric, symbol Device:R
- added R306, R307, R308: 1k, Resistor_SMD:R_0402_1005Metric, symbol Device:R_US
- added SW201: RESET, lzptr:SW_TL3365AF180QG, symbol Switch:SW_SPST
- added SW202: BOOTSEL, lzptr:SW_TL3365AF180QG, symbol Switch:SW_SPST
- added U203: W25Q128JVS, Package_SO:SOIC-8_5.23x5.23mm_P1.27mm, symbol Memory_Flash:W25Q128JVS
- renumbered C216 to C201, C215 to C202, C201 to C203, C202 to C204, C203 to C205, C204 to C206, C205 to C207, C206 to C208, C207 to C209, C209 to C210, C210 to C211, C211 to C212, C212 to C213, C208 to C215, C213 to C216, D205 to D204, L202 to L201, R201 to R203, R207 to R206, R213 to R207, R214 to R208, U104 to U201
Connections:
- net +3.3V: now also U201.44 (VREG_IN), C217.1, C218.1, R212.2, U203.8 (VCC); no longer C203.1, C204.1, C205.1, U201.23 (DVDD), U201.45 (VREG_VOUT), U201.50 (DVDD)
- net GND: now also C217.2, C218.2, R306.1, R307.1, R308.2, U203.4 (GND)
- net RUN: now also U201.26 (RUN), SW201.1 (A)
- net USB_D+: now also R201.1
- net USB_D-: now also R202.1
- net ACT_LED: now reaches U201.2 (GPIO0)
- net ACT_LED: now also D301.2 (A)
- net DAC_NLDAC: now reaches U201.27 (GPIO16)
- net DAC_NCLR: now reaches U201.28 (GPIO17)
- net DAC_SPI0_CLK: now reaches U201.29 (GPIO18)
- net DAC_SPI0_MOSI: now reaches U201.30 (GPIO19)
- net DAC_SPI0_NCS: now reaches U201.32 (GPIO21)
- net ADC_SPI1_CLK: now reaches U201.34 (GPIO22)
- net ADC_SPI1_MISO: now reaches U201.36 (GPIO24)
- net ADC_SPI1_NCS: now reaches U201.37 (GPIO25)
- net USB_DT-: now reaches U201.46 (USB_DM)
- net USB_DT-: now also R202.2
- net USB_DT+: now reaches U201.47 (USB_DP)
- net USB_DT+: now also R201.2
- net QSPI_SD3: now reaches U201.51 (QSPI_SD3)
- net QSPI_SD3: now also U203.7 (IO3)
- net QSPI_SCLK: now reaches U201.52 (QSPI_SCLK)
- net QSPI_SCLK: now also U203.6 (CLK)
- net QSPI_SD0: now reaches U201.53 (QSPI_SD0)
- net QSPI_SD0: now also U203.5 (DI(IO0))
- net QSPI_SD2: now reaches U201.54 (QSPI_SD2)
- net QSPI_SD2: now also U203.3 (IO2)
- net QSPI_SD1: now reaches U201.55 (QSPI_SD1)
- net QSPI_SD1: now also U203.2 (DO(IO1))
- net QSPI_CS: now reaches U201.56 (QSPI_SS)
- net QSPI_CS: now also R212.1, SW202.1 (A), U203.1 (~{CS})
- new net: D301.1 (K), R308.1
- new net: R306.2, SW201.2 (B)
- new net: R307.2, SW202.2 (B)
- new net +1V1: C203.1, C204.1, C205.1, U201.23 (DVDD), U201.45 (VREG_VOUT), U201.50 (DVDD)
- no-connect marks 6 -> 27
Other:
- note added: "QSPI Flash"
- note added: "Reset, Bootsel, LEDS"
- moved on the sheet: C203, C204, C205, C206, C207, C208, C209, C210, C211, C212, C213, C214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

Commit message: Finished rp2040 schematic
Connections:
- net ADC_SPI1_CLK: now also U201.29 (GPIO18); no longer U201.34 (GPIO22)
- net ADC_SPI1_MISO: now also U201.31 (GPIO20); no longer U201.36 (GPIO24)
- net ADC_SPI1_NCS: now also U201.32 (GPIO21); no longer U201.37 (GPIO25)
- net DAC_NCLR: now also U201.39 (GPIO27_ADC1); no longer U201.28 (GPIO17)
- net DAC_NLDAC: now also U201.38 (GPIO26_ADC0); no longer U201.27 (GPIO16)
- net DAC_SPI0_CLK: now also U201.34 (GPIO22); no longer U201.29 (GPIO18)
- net DAC_SPI0_MOSI: now also U201.35 (GPIO23); no longer U201.30 (GPIO19)
- net DAC_SPI0_NCS: now also U201.37 (GPIO25); no longer U201.32 (GPIO21)
- net XOUT: now reaches R203.2, U201.21 (XOUT)
- net XIN: now reaches C201.1, U201.20 (XIN), Y201.1
Changed lines of the file:
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@@
   (no_connect (at 181.61 130.81))
   (no_connect (at 48.26 173.99))
-  (no_connect (at 110.49 120.65))
   (no_connect (at 110.49 57.15))
   (no_connect (at 35.56 173.99))
   (no_connect (at 110.49 82.55))
   (no_connect (at 110.49 74.93))
+  (no_connect (at 110.49 110.49))
   (no_connect (at 110.49 62.23))
   (no_connect (at 110.49 80.01))
@@
   (no_connect (at 110.49 77.47))
   (no_connect (at 110.49 123.19))
+  (no_connect (at 110.49 97.79))
   (no_connect (at 110.49 85.09))
+  (no_connect (at 110.49 92.71))
   (no_connect (at 110.49 54.61))
   (no_connect (at 48.26 171.45))
-  (no_connect (at 110.49 100.33))
-  (no_connect (at 110.49 107.95))
   (no_connect (at 110.49 59.69))
-  (no_connect (at 110.49 118.11))
+  (no_connect (at 110.49 90.17))
   (no_connect (at 158.75 138.43))
   (no_connect (at 110.49 69.85))
@@
     (stroke (width 0) (type default))
   )
-  (wire (pts (xy 110.49 90.17) (xy 114.3 90.17))
-    (stroke (width 0) (type default))
-  )
   (wire (pts (xy 92.71 41.91) (xy 92.71 40.64))
     (stroke (width 0) (type default))
@@
     (stroke (width 0) (type default))
   )
-  (wire (pts (xy 110.49 113.03) (xy 114.3 113.03))
-    (stroke (width 0) (type default))
-  )
   (wire (pts (xy 80.01 41.91) (xy 80.01 40.64))
     (stroke (width 0) (type default))
@@
     (stroke (width 0) (type default))
   )
-  (wire (pts (xy 114.3 95.25) (xy 110.49 95.25))
-    (stroke (width 0) (type default))
-  )
   (wire (pts (xy 36.83 123.19) (xy 36.83 130.81))
     (stroke (width 0) (type default))
@@
     (stroke (width 0) (type default))
   )
+  (wire (pts (xy 110.49 120.65) (xy 115.57 120.65))
+    (stroke (width 0) (type default))
+  )
   (wire (pts (xy 100.33 31.75) (xy 113.03 31.75))
     (stroke (width 0) (type default))
@@
     (stroke (width 0) (type default))
   )
-  (wire (pts (xy 110.49 110.49) (xy 114.3 110.49))
-    (stroke (width 0) (type default))
-  )
   (wire (pts (xy 33.02 179.07) (xy 26.67 179.07))
     (stroke (width 0) (type default))
   )
-  (wire (pts (xy 110.49 97.79) (xy 114.3 97.79))
-    (stroke (width 0) (type default))
-  )
   (wire (pts (xy 176.53 21.59) (xy 189.23 21.59))
     (stroke (width 0) (type default))
@@
     (stroke (width 0) (type default))
   )
+  (wire (pts (xy 110.49 100.33) (xy 115.57 100.33))
+    (stroke (width 0) (type default))
+  )
   (wire (pts (xy 229.87 62.23) (xy 231.14 62.23))
     (stroke (width 0) (type default))
@@
     (stroke (width 0) (type default))
   )
+  (wire (pts (xy 110.49 113.03) (xy 115.57 113.03))
+    (stroke (width 0) (type default))
+  )
   (wire (pts (xy 125.73 21.59) (xy 138.43 21.59))
     (stroke (width 0) (type default))
@@
     (stroke (width 0) (type default))
   )
+  (wire (pts (xy 110.49 118.11) (xy 115.57 118.11))
+    (stroke (width 0) (type default))
+  )
   (wire (pts (xy 66.04 30.48) (xy 66.04 31.75))
     (stroke (width 0) (type default))
@@
     (stroke (width 0) (type default))
   )
+  (wire (pts (xy 110.49 105.41) (xy 115.57 105.41))
+    (stroke (width 0) (type default))
+  )
   (wire (pts (xy 62.23 186.69) (xy 62.23 187.96))
     (stroke (width 0) (type default))
@@
     (stroke (width 0) (type default))
   )
-  (wire (pts (xy 110.49 105.41) (xy 114.3 105.41))
+  (wire (pts (xy 110.49 95.25) (xy 115.57 95.25))
     (stroke (width 0) (type default))
   )
@@
     (stroke (width 0) (type default))
   )
+  (wire (pts (xy 110.49 107.95) (xy 115.57 107.95))
+    (stroke (width 0) (type default))
+  )
   (wire (pts (xy 229.87 52.07) (xy 229.87 50.8))
     (stroke (width 0) (type default))
@@
     (stroke (width 0) (type default))
   )
+  (wire (pts (xy 110.49 102.87) (xy 115.57 102.87))
+    (stroke (width 0) (type default))
+  )
   (wire (pts (xy 24.13 95.25) (xy 24.13 115.57))
     (stroke (width 0) (type default))
@@
     (stroke (width 0) (type default))
   )
-  (wire (pts (xy 114.3 102.87) (xy 110.49 102.87))
-    (stroke (width 0) (type default))
-  )
   (wire (pts (xy 215.9 69.85) (xy 231.14 69.85))
     (stroke (width 0) (type default))
@@
   )
   (wire (pts (xy 100.33 30.48) (xy 100.33 31.75))
-    (stroke (width 0) (type default))
-  )
-  (wire (pts (xy 110.49 92.71) (xy 114.3 92.71))
     (stroke (width 0) (type default))
   )
@@
     (effects (font (size 1.27 1.27)) (justify left bottom))
   )
+  (label "XIN" (at 55.88 95.25 0) (fields_autoplaced)
+    (effects (font (size 1.27 1.27)) (justify left bottom))
+  )
   (label "USB_D+" (at 27.94 57.15 0) (fields_autoplaced)
     (effects (font (size 1.27 1.27)) (justify left bottom))
@@
     (effects (font (size 1.27 1.27)) (justify right bottom))
   )
+  (label "XOUT" (at 54.61 105.41 0) (fields_autoplaced)
+    (effects (font (size 1.27 1.27)) (justify left bottom))
+  )
   (label "USB_CONN_D+" (at 273.05 113.03 180) (fields_autoplaced)
     (effects (font (size 1.27 1.27)) (justify right bottom))
@@
     (effects (font (size 1.27 1.27)) (justify left bottom))
   )
-  (hierarchical_label "ADC_SPI1_CLK" (shape output) (at 114.3 105.41 0) (fields_autoplaced)
+  (hierarchical_label "ADC_SPI1_CLK" (shape output) (at 115.57 95.25 0) (fields_autoplaced)
     (effects (font (size 1.27 1.27)) (justify left))
   )
-  (hierarchical_label "ADC_SPI1_MISO" (shape input) (at 114.3 110.49 0) (fields_autoplaced)
+  (hierarchical_label "ADC_SPI1_MISO" (shape input) (at 115.57 100.33 0) (fields_autoplaced)
     (effects (font (size 1.27 1.27)) (justify left))
   )
-  (hierarchical_label "DAC_NLDAC" (shape output) (at 114.3 90.17 0) (fields_autoplaced)
+  (hierarchical_label "DAC_NLDAC" (shape output) (at 115.57 118.11 0) (fields_autoplaced)
     (effects (font (size 1.27 1.27)) (justify left))
   )
-  (hierarchical_label "DAC_SPI0_CLK" (shape output) (at 114.3 95.25 0) (fields_autoplaced)
+  (hierarchical_label "DAC_SPI0_CLK" (shape output) (at 115.57 105.41 0) (fields_autoplaced)
     (effects (font (size 1.27 1.27)) (justify left))
   )
-  (hierarchical_label "DAC_NCLR" (shape output) (at 114.3 92.71 0) (fields_autoplaced)
+  (hierarchical_label "DAC_NCLR" (shape output) (at 115.57 120.65 0) (fields_autoplaced)
     (effects (font (size 1.27 1.27)) (justify left))
   )
-  (hierarchical_label "DAC_SPI0_NCS" (shape output) (at 114.3 102.87 0) (fields_autoplaced)
+  (hierarchical_label "DAC_SPI0_NCS" (shape output) (at 115.57 113.03 0) (fields_autoplaced)
     (effects (font (size 1.27 1.27)) (justify left))
   )
-  (hierarchical_label "DAC_SPI0_MOSI" (shape output) (at 114.3 97.79 0) (fields_autoplaced)
+  (hierarchical_label "DAC_SPI0_MOSI" (shape output) (at 115.57 107.95 0) (fields_autoplaced)
     (effects (font (size 1.27 1.27)) (justify left))
   )
-  (hierarchical_label "ADC_SPI1_NCS" (shape output) (at 114.3 113.03 0) (fields_autoplaced)
+  (hierarchical_label "ADC_SPI1_NCS" (shape output) (at 115.57 102.87 0) (fields_autoplaced)
     (effects (font (size 1.27 1.27)) (justify left))
   )

Commit message: Finished layout changes
Parts:
- removed C214: 100n, Capacitor_SMD:C_0402_1005Metric, symbol Device:C
- C201, C202: Rating 10V -> 5% 10V
- C205, C206: Rating (none) -> 10V
- C216: renamed from C217; Rating (none) -> 10V
- R212: now left out of the parts list
- renumbered C215 to C214, C216 to C215, C218 to C217
Connections:
- net ACT_LED: now also U201.41 (GPIO29_ADC3); no longer U201.2 (GPIO0)
- net CR_XOUT: now reaches C202.1, R203.1, Y201.3
Other:
- moved on the sheet: Y201

Commit message: Finished routing
Parts:
- C203, C204, C207, C208, C209, C210, C211, C212, C213, C215, C217: MPN CC0402KRX5R6BB104 -> C1525; Rating 10V -> 16V
- C205, C206, C216: MPN (none) -> C52923; Rating 10V -> 25V
Connections:
- net ACT_LED: now also U201.14 (GPIO11); no longer U201.41 (GPIO29_ADC3)
- net CONN_SWCLK: now also D202.1 (A1), J201.2 (Pin_2), R204.2; no longer D203.1 (A1), J201.4 (Pin_4), R205.2
- net CONN_SWDIO: now also D203.1 (A1), J201.4 (Pin_4), R205.2; no longer D202.1 (A1), J201.2 (Pin_2), R204.2
- net SWCLK: now also R204.1; no longer R205.1
- net SWDIO: now also R205.1; no longer R204.1

Commit message: Finished bom
Parts:
- C201, C202: MPN CC0402KRX5R6BB104 -> C1570; Rating 5% 10V -> 5% 50V
- C205, C206, C216: Rating 25V -> 50V
- C214: MPN CC0402KRX5R6BB104 -> C1525; Rating 10V -> 16V
- D201, D202, D203, D204: MPN (none) -> C51450; Rating (none) -> 5.8V 26V
- D301: MPN (none) -> C2292
- J201: MPN (none) -> C598540
- J202: MPN (none) -> C165948
- L201: MPN (none) -> C963740; Rating (none) -> 90Ω@100MHz
- R201, R202: MPN (none) -> C321419
- R203, R306, R307, R308: MPN (none) -> C11702
- R204, R205, R206: MPN (none) -> C25120
- R207, R208: MPN (none) -> C25905
- R212: value 10k -> DNP 10k; Rating (none) -> 63mW
- SW201, SW202: MPN (none) -> C2886926
- U201: MPN (none) -> C2040
- U202: MPN (none) -> C5261088
- U203: MPN C113767 -> C97521
- Y201: MPN (none) -> C9002
Connections:
- net CONN_SWCLK: now also D203.1 (A1), J201.4 (Pin_4), R205.2; no longer D202.1 (A1), J201.2 (Pin_2), R204.2
- net CONN_SWDIO: now also D202.1 (A1), J201.2 (Pin_2), R204.2; no longer D203.1 (A1), J201.4 (Pin_4), R205.2
- net SWCLK: now also R205.1; no longer R204.1
- net SWDIO: now also R204.1; no longer R205.1
Changed lines of the file:
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@@
     (effects (font (size 1.27 1.27)) (justify right bottom))
   )
-  (label "CONN_SWDIO" (at 67.31 168.91 0) (fields_autoplaced)
+  (label "CONN_SWCLK" (at 67.31 168.91 0) (fields_autoplaced)
     (effects (font (size 1.27 1.27)) (justify left bottom))
   )
@@
     (effects (font (size 1.27 1.27)) (justify left bottom))
   )
-  (label "SWCLK" (at 107.95 166.37 180) (fields_autoplaced)
+  (label "SWDIO" (at 107.95 166.37 180) (fields_autoplaced)
     (effects (font (size 1.27 1.27)) (justify right bottom))
   )
@@
     (effects (font (size 1.27 1.27)) (justify left bottom))
   )
-  (label "SWDIO" (at 107.95 168.91 180) (fields_autoplaced)
+  (label "SWCLK" (at 107.95 168.91 180) (fields_autoplaced)
     (effects (font (size 1.27 1.27)) (justify right bottom))
   )
@@
     (effects (font (size 1.27 1.27)) (justify left bottom))
   )
-  (label "CONN_SWCLK" (at 67.31 166.37 0) (fields_autoplaced)
+  (label "CONN_SWDIO" (at 67.31 166.37 0) (fields_autoplaced)
     (effects (font (size 1.27 1.27)) (justify left bottom))
   )
@@
       (effects (font (size 1.27 1.27)) (justify left))
     )
-    (property "MPN" "" (at 46.99 59.69 0)
+    (property "MPN" "C321419" (at 46.99 59.69 0)
       (effects (font (size 1.27 1.27)) hide)
     )
@@
   (symbol (lib_id "Device:R") (at 229.87 55.88 0) (mirror x) (unit 1)
     (in_bom no) (on_board yes) (dnp yes)
-    (property "Reference" "R212" (at 222.25 54.61 0)
-      (effects (font (size 1.27 1.27)) (justify left))
-    )
-    (property "Value" "10k" (at 223.52 57.15 0)
+    (property "Reference" "R212" (at 219.71 54.61 0)
+      (effects (font (size 1.27 1.27)) (justify left))
+    )
+    (property "Value" "DNP 10k" (at 219.71 57.15 0)
       (effects (font (size 1.27 1.27)) (justify left))
     )
@@
       (effects (font (size 1.27 1.27)) hide)
     )
-    (property "Rating" "" (at 229.87 52.07 90)
+    (property "Rating" "63mW" (at 229.87 52.07 90)
       (effects (font (size 1.27 1.27)) (justify left))
     )
@@
     )
     (property "Datasheet" "~" (at 40.64 171.45 0)
+      (effects (font (size 1.27 1.27)) hide)
+    )
+    (property "MPN" "C598540" (at 40.64 171.45 0)
       (effects (font (size 1.27 1.27)) hide)
     )
@@
       (effects (font (size 1.27 1.27)) hide)
     )
+    (property "MPN" "C51450" (at 82.55 182.88 0)
+      (effects (font (size 1.27 1.27)) hide)
+    )
+    (property "Rating" "5.8V 26V" (at 82.55 182.88 0)
+      (effects (font (size 1.27 1.27)) hide)
+    )
     (pin "1")
     (pin "2")
@@
       (effects (font (size 1.27 1.27)) (justify left))
     )
-    (property "MPN" "" (at 46.99 57.15 0)
+    (property "MPN" "C321419" (at 46.99 57.15 0)
       (effects (font (size 1.27 1.27)) hide)
     )
@@
       (effects (font (size 1.27 1.27)) (justify left))
     )
+    (property "MPN" "C11702" (at 50.8 105.41 0)
+      (effects (font (size 1.27 1.27)) hide)
+    )
     (pin "1")
     (pin "2")
@@
       (effects (font (size 1.27 1.27)) (justify left))
     )
+    (property "MPN" "C25905" (at 207.01 104.14 0)
+      (effects (font (size 1.27 1.27)) hide)
+    )
     (pin "1")
     (pin "2")
@@
       (effects (font (size 1.27 1.27)))
     )
-    (property "MPN" "" (at 85.09 87.63 0)
+    (property "MPN" "C2040" (at 85.09 87.63 0)
       (effects (font (size 1.27 1.27)) hide)
     )
@@
       (effects (font (size 1.27 1.27)) hide)
     )
-    (property "MPN" "CC0402KRX5R6BB104" (at 24.13 123.19 0)
-      (effects (font (size 1.27 1.27)) hide)
-    )
-    (property "Rating" "5% 10V" (at 19.05 127 0)
+    (property "MPN" "C1570" (at 24.13 123.19 0)
+      (effects (font (size 1.27 1.27)) hide)
+    )
+    (property "Rating" "5% 50V" (at 19.05 127 0)
       (effects (font (size 1.27 1.27)))
     )
@@
     (property "Rating" "63mW" (at 210.82 109.22 90)
       (effects (font (size 1.27 1.27)) (justify left))
+    )
+    (property "MPN" "C25905" (at 207.01 109.22 0)
+      (effects (font (size 1.27 1.27)) hide)
     )
     (pin "1")
@@
     )
     (property "LCSC Parrt #" "" (at 247.65 110.49 0)
+      (effects (font (size 1.27 1.27)) hide)
+    )
+    (property "MPN" "C5261088" (at 247.65 110.49 0)
       (effects (font (size 1.27 1.27)) hide)
     )
@@
       (effects (font (size 1.27 1.27)) hide)
     )
-    (property "Datasheet" "https://www.usb.org/sites/default/files/documents/usb_type-c.zip" (at 170.18 115.57 0)
+    (property "Datasheet" "~" (at 170.18 115.57 0)
+      (effects (font (size 1.27 1.27)) hide)
+    )
+    (property "MPN" "C165948" (at 166.37 115.57 0)
       (effects (font (size 1.27 1.27)) hide)
     )
@@
       (effects (font (size 1.27 1.27)) hide)
     )
-    (property "Rating" "25V" (at 69.85 30.48 0)
+    (property "Rating" "50V" (at 69.85 30.48 0)
       (effects (font (size 1.27 1.27)) (justify left))
     )
@@
       (effects (font (size 1.27 1.27)) (justify right))
     )
-    (property "MPN" "" (at 187.96 60.96 0)
+    (property "MPN" "C2292" (at 187.96 60.96 0)
       (effects (font (size 1.27 1.27)) hide)
     )
@@
       (effects (font (size 1.27 1.27)) hide)
     )
+    (property "MPN" "C51450" (at 52.07 182.88 0)
+      (effects (font (size 1.27 1.27)) hide)
+    )
+    (property "Rating" "5.8V 26V" (at 52.07 182.88 0)
+      (effects (font (size 1.27 1.27)) hide)
+    )
     (pin "1")
     (pin "2")
@@
       (effects (font (size 1.27 1.27)))
     )
+    (property "MPN" "C25120" (at 91.44 176.53 0)
+      (effects (font (size 1.27 1.27)) hide)
+    )
     (pin "1")
     (pin "2")
@@
       (effects (font (size 1.27 1.27)) hide)
     )
-    (property "Rating" "25V" (at 255.27 60.96 0)
+    (property "Rating" "50V" (at 255.27 60.96 0)
       (effects (font (size 1.27 1.27)) (justify left))
     )
@@
       (effects (font (size 1.27 1.27)) hide)
     )
+    (property "MPN" "C51450" (at 26.67 172.72 0)
+      (effects (font (size 1.27 1.27)) hide)
+    )
+    (property "Rating" "5.8V 26V" (at 26.67 172.72 0)
+      (effects (font (size 1.27 1.27)) hide)
+    )
     (pin "1")
     (pin "2")
@@
       (effects (font (size 1.27 1.27)))
     )
-    (property "MPN" "" (at 148.59 64.77 0)
+    (property "MPN" "C2886926" (at 148.59 64.77 0)
       (effects (font (size 1.27 1.27)) hide)
     )
@@
       (effects (font (size 1.27 1.27)))
     )
-    (property "MPN" "" (at 168.91 64.77 0)
+    (property "MPN" "C2886926" (at 168.91 64.77 0)
       (effects (font (size 1.27 1.27)) hide)
     )
@@
     (property "Rating" "63mW" (at 91.44 166.37 90)
       (effects (font (size 1.27 1.27)))
+    )
+    (property "MPN" "C25120" (at 91.44 166.37 0)
+      (effects (font (size 1.27 1.27)) hide)
     )
     (pin "1")
@@
       (effects (font (size 1.27 1.27)) hide)
     )
+    (property "MPN" "C51450" (at 62.23 182.88 0)
+      (effects (font (size 1.27 1.27)) hide)
+    )
+    (property "Rating" "5.8V 26V" (at 62.23 182.88 0)
+      (effects (font (size 1.27 1.27)) hide)
+    )
     (pin "1")
     (pin "2")
@@
       (effects (font (size 1.27 1.27)) hide)
     )
-    (property "MPN" "CC0402KRX5R6BB104" (at 101.6 182.88 0)
-      (effects (font (size 1.27 1.27)) hide)
-    )
-    (property "Rating" "10V" (at 107.95 186.69 0)
+    (property "MPN" "C1525" (at 101.6 182.88 0)
+      (effects (font (size 1.27 1.27)) hide)
+    )
+    (property "Rating" "16V" (at 107.95 186.69 0)
       (effects (font (size 1.27 1.27)))
     )
@@
       (effects (font (size 1.27 1.27)) hide)
     )
-    (property "MPN" "CC0402KRX5R6BB104" (at 45.72 123.19 0)
-      (effects (font (size 1.27 1.27)) hide)
-    )
-    (property "Rating" "5% 10V" (at 53.34 127 0)
+    (property "MPN" "C1570" (at 45.72 123.19 0)
+      (effects (font (size 1.27 1.27)) hide)
+    )
+    (property "Rating" "5% 50V" (at 53.34 127 0)
       (effects (font (size 1.27 1.27)))
     )
@@
       (effects (font (size 1.27 1.27)))
     )
-    (property "MPN" "C113767" (at 241.3 69.85 0)
+    (property "MPN" "C97521" (at 241.3 69.85 0)
       (effects (font (size 1.27 1.27)) hide)
     )
@@
       (effects (font (size 1.27 1.27)) hide)
     )
-    (property "Rating" "25V" (at 104.14 30.48 0)
+    (property "Rating" "50V" (at 104.14 30.48 0)
       (effects (font (size 1.27 1.27)) (justify left))
     )
@@
       (effects (font (size 1.27 1.27)) (justify left))
     )
-    (property "MPN" "" (at 187.96 73.66 0)
+    (property "MPN" "C11702" (at 187.96 73.66 0)
       (effects (font (size 1.27 1.27)) hide)
     )
@@
       (effects (font (size 1.27 1.27)) (justify left))
     )
-    (property "MPN" "" (at 148.59 73.66 0)
+    (property "MPN" "C11702" (at 148.59 73.66 0)
       (effects (font (size 1.27 1.27)) hide)
     )
@@
       (effects (font (size 1.27 1.27)) (justify left))
     )
-    (property "MPN" "" (at 168.91 73.66 0)
+    (property "MPN" "C11702" (at 168.91 73.66 0)
       (effects (font (size 1.27 1.27)) hide)
     )
@@
       (effects (font (size 1.27 1.27)) hide)
     )
+    (property "MPN" "C963740" (at 247.65 133.35 0)
+      (effects (font (size 1.27 1.27)) hide)
+    )
+    (property "Rating" "90Ω@100MHz " (at 247.65 133.35 0)
+      (effects (font (size 1.27 1.27)) hide)
+    )
     (pin "1")
     (pin "2")
@@
       (effects (font (size 1.27 1.27)))
     )
+    (property "MPN" "C25120" (at 91.44 168.91 0)
+      (effects (font (size 1.27 1.27)) hide)
+    )
     (pin "1")
     (pin "2")
@@
       (effects (font (size 1.27 1.27)))
     )
-    (property "MPN" "" (at 33.02 115.57 0)
-      (effects (font (size 1.27 1.27)) hide)
-    )
+    (property "MPN" "C9002" (at 33.02 115.57 0)
+      (effects (font (size 1.27 1.27)) hide)
+    )
