File: hardware/mcu.kicad_sch (KiCad schematic)
At the start: 43 parts, among them J201 2x5 1.27mm, J202 USB_C_Receptacle_USB2.0, SW201 RESET, SW202 BOOTSEL, U201 RP2040, U202 USBLC6-2SC6, U203 W25Q128JVS, Y201 Crystal_GND24

Commit message: Cleanup, minor bom changes and finished production files
Parts:
- D201, D202, D203, D204: value PESD3V3L1BA,115 -> PESD3V3L1BA; MPN C51450 -> C2939000; Rating 5.8V 26V -> 4V 10.5V
- D301: MPN C2292 -> C72043
Changed lines of the file:
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@@
       (effects (font (size 1.27 1.27)) (justify left))
     )
-    (property "Value" "PESD3V3L1BA,115" (at 85.09 190.5 90)
+    (property "Value" "PESD3V3L1BA" (at 85.09 190.5 90)
       (effects (font (size 1.27 1.27)) (justify left) hide)
     )
@@
       (effects (font (size 1.27 1.27)) hide)
     )
-    (property "MPN" "C51450" (at 82.55 182.88 0)
-      (effects (font (size 1.27 1.27)) hide)
-    )
-    (property "Rating" "5.8V 26V" (at 82.55 182.88 0)
+    (property "MPN" "C2939000" (at 82.55 182.88 0)
+      (effects (font (size 1.27 1.27)) hide)
+    )
+    (property "Rating" "4V 10.5V" (at 82.55 182.88 0)
       (effects (font (size 1.27 1.27)) hide)
     )
@@
       (effects (font (size 1.27 1.27)) (justify right))
     )
-    (property "MPN" "C2292" (at 187.96 60.96 0)
+    (property "MPN" "C72043" (at 187.96 60.96 0)
       (effects (font (size 1.27 1.27)) hide)
     )
@@
       (effects (font (size 1.27 1.27)) (justify left))
     )
-    (property "Value" "PESD3V3L1BA,115" (at 58.42 190.5 90)
+    (property "Value" "PESD3V3L1BA" (at 58.42 190.5 90)
       (effects (font (size 1.27 1.27)) (justify left))
     )
@@
       (effects (font (size 1.27 1.27)) hide)
     )
-    (property "MPN" "C51450" (at 52.07 182.88 0)
-      (effects (font (size 1.27 1.27)) hide)
-    )
-    (property "Rating" "5.8V 26V" (at 52.07 182.88 0)
+    (property "MPN" "C2939000" (at 52.07 182.88 0)
+      (effects (font (size 1.27 1.27)) hide)
+    )
+    (property "Rating" "4V 10.5V" (at 52.07 182.88 0)
       (effects (font (size 1.27 1.27)) hide)
     )
@@
       (effects (font (size 1.27 1.27)) (justify left))
     )
-    (property "Value" "PESD3V3L1BA,115" (at 17.78 185.42 90)
+    (property "Value" "PESD3V3L1BA" (at 17.78 185.42 90)
       (effects (font (size 1.27 1.27)) (justify left))
     )
@@
       (effects (font (size 1.27 1.27)) hide)
     )
-    (property "MPN" "C51450" (at 26.67 172.72 0)
-      (effects (font (size 1.27 1.27)) hide)
-    )
-    (property "Rating" "5.8V 26V" (at 26.67 172.72 0)
+    (property "MPN" "C2939000" (at 26.67 172.72 0)
+      (effects (font (size 1.27 1.27)) hide)
+    )
+    (property "Rating" "4V 10.5V" (at 26.67 172.72 0)
       (effects (font (size 1.27 1.27)) hide)
     )
@@
       (effects (font (size 1.27 1.27)) (justify left))
     )
-    (property "Value" "PESD3V3L1BA,115" (at 64.77 190.5 90)
+    (property "Value" "PESD3V3L1BA" (at 64.77 190.5 90)
       (effects (font (size 1.27 1.27)) (justify left) hide)
     )
@@
       (effects (font (size 1.27 1.27)) hide)
     )
-    (property "MPN" "C51450" (at 62.23 182.88 0)
-      (effects (font (size 1.27 1.27)) hide)
-    )
-    (property "Rating" "5.8V 26V" (at 62.23 182.88 0)
-      (effects (font (size 1.27 1.27)) hide)
-    )
+    (property "MPN" "C2939000" (at 62.23 182.88 0)
+      (effects (font (size 1.27 1.27)) hide)
+    )
+    (property "Rating" "4V 10.5V" (at 62.23 182.88 0)
+      (effects (font (size 1.27 1.27)) hide)
+    )

Commit message: Fixed missing pull up for run pin
Parts:
- added R402: 10k, Resistor_SMD:R_0402_1005Metric, symbol Device:R
- R306, R307, R308: symbol Device:R_US -> Device:R
Connections:
- net +3.3V: now also R402.1
- net RUN: now also R402.2
Changed lines of the file:
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@@
     (title "RP2040 Audio Board")
     (date "2023-05-01")
-    (rev "0.1")
+    (rev "0.2")
     (company "LP")
   )
@@
     (stroke (width 0) (type default))
   )
+  (wire (pts (xy 34.29 49.53) (xy 29.21 49.53))
+    (stroke (width 0) (type default))
+  )
   (wire (pts (xy 82.55 40.64) (xy 80.01 40.64))
     (stroke (width 0) (type default))
@@
     (stroke (width 0) (type default))
   )
+  (wire (pts (xy 41.91 49.53) (xy 59.69 49.53))
+    (stroke (width 0) (type default))
+  )
   (polyline (pts (xy 15.24 153.67) (xy 15.24 194.31))
     (stroke (width 0) (type default))
@@
     (stroke (width 0) (type default))
   )
-  (wire (pts (xy 44.45 49.53) (xy 59.69 49.53))
-    (stroke (width 0) (type default))
-  )
   (wire (pts (xy 265.43 60.96) (xy 265.43 62.23))
     (stroke (width 0) (type default))
@@
   )
   (wire (pts (xy 181.61 105.41) (xy 196.85 105.41))
+    (stroke (width 0) (type default))
+  )
+  (wire (pts (xy 29.21 49.53) (xy 29.21 46.99))
     (stroke (width 0) (type default))
   )
@@
     )
   )
+  (symbol (lib_id "power:+3.3V") (at 29.21 46.99 0) (unit 1)
+    (in_bom yes) (on_board yes) (dnp no)
+    (property "Reference" "#PWR0115" (at 29.21 50.8 0)
+      (effects (font (size 1.27 1.27)) hide)
+    )
+    (property "Value" "+3.3V" (at 29.21 43.18 0)
+      (effects (font (size 1.27 1.27)))
+    )
+    (property "Footprint" "" (at 29.21 46.99 0)
+      (effects (font (size 1.27 1.27)) hide)
+    )
+    (property "Datasheet" "" (at 29.21 46.99 0)
+      (effects (font (size 1.27 1.27)) hide)
+    )
+    (pin "1")
+    (instances
+      (project "rp2040_audioboard"
+        (path "/ef85fc54-329f-434a-8339-262c7e24e2e9/8b86c5bb-c0fc-4d5a-91aa-2ce0ad602b27"
+          (reference "#PWR0115") (unit 1)
+        )
+        (path "/ef85fc54-329f-434a-8339-262c7e24e2e9/ee2d4daf-adb5-47d0-ba60-e54b60815215"
+          (reference "#PWR0221") (unit 1)
+        )
+      )
+    )
+  )
   (symbol (lib_id "Device:C") (at 163.83 26.67 0) (unit 1)
     (in_bom yes) (on_board yes) (dnp no)
@@
     )
   )
-  (symbol (lib_id "Device:R_US") (at 187.96 73.66 0) (unit 1)
+  (symbol (lib_id "Device:R") (at 187.96 73.66 0) (unit 1)
     (in_bom yes) (on_board yes) (dnp no) (fields_autoplaced)
     (property "Reference" "R308" (at 189.865 71.1199 0)
@@
       (effects (font (size 1.27 1.27)) (justify left))
     )
-    (property "Footprint" "Resistor_SMD:R_0402_1005Metric" (at 188.976 73.914 90)
+    (property "Footprint" "Resistor_SMD:R_0402_1005Metric" (at 186.182 73.66 90)
       (effects (font (size 1.27 1.27)) hide)
     )
@@
     )
   )
-  (symbol (lib_id "Device:R_US") (at 148.59 73.66 180) (unit 1)
+  (symbol (lib_id "Device:R") (at 148.59 73.66 180) (unit 1)
     (in_bom yes) (on_board yes) (dnp no) (fields_autoplaced)
     (property "Reference" "R306" (at 146.05 71.1199 0)
@@
       (effects (font (size 1.27 1.27)) (justify left))
     )
-    (property "Footprint" "Resistor_SMD:R_0402_1005Metric" (at 147.574 73.406 90)
+    (property "Footprint" "Resistor_SMD:R_0402_1005Metric" (at 150.368 73.66 90)
       (effects (font (size 1.27 1.27)) hide)
     )
@@
     )
   )
-  (symbol (lib_id "Device:R_US") (at 168.91 73.66 180) (unit 1)
+  (symbol (lib_id "Device:R") (at 168.91 73.66 180) (unit 1)
     (in_bom yes) (on_board yes) (dnp no) (fields_autoplaced)
     (property "Reference" "R307" (at 167.005 71.1199 0)
@@
       (effects (font (size 1.27 1.27)) (justify left))
     )
-    (property "Footprint" "Resistor_SMD:R_0402_1005Metric" (at 167.894 73.406 90)
+    (property "Footprint" "Resistor_SMD:R_0402_1005Metric" (at 170.688 73.66 90)
       (effects (font (size 1.27 1.27)) hide)
     )
@@
         )
       )
+    )
+  )
+  (symbol (lib_id "Device:R") (at 38.1 49.53 90) (unit 1)
+    (in_bom yes) (on_board yes) (dnp no)
+    (property "Reference" "R402" (at 40.64 46.99 90)
+      (effects (font (size 1.27 1.27)) (justify left))
+    )
+    (property "Value" "10k" (at 39.37 52.07 90)
+      (effects (font (size 1.27 1.27)) (justify left))
+    )
+    (property "Footprint" "Resistor_SMD:R_0402_1005Metric" (at 38.1 51.308 90)
+      (effects (font (size 1.27 1.27)) hide)
+    )
+    (property "Datasheet" "~" (at 38.1 49.53 0)
+      (effects (font (size 1.27 1.27)) hide)
+    )
+    (property "Rating" "63mW" (at 41.91 49.53 90)
+      (effects (font (size 1.27 1.27)) (justify left))
+    )
+    (property "MPN" "C25744" (at 38.1 49.53 0)
+      (effects (font (size 1.27 1.27)) hide)
+    )
+    (pin "1")
+    (pin "2")
+    (instances
+      (project "rp2040_audioboard"
+        (path "/ef85fc54-329f-434a-8339-262c7e24e2e9/a834fb14-b3a1-4fa1-8c02-1fdc386616f0"
+          (reference "R402") (unit 1)
+        )
+        (path "/ef85fc54-329f-434a-8339-262c7e24e2e9/ee2d4daf-adb5-47d0-ba60-e54b60815215"
+          (reference "R213") (unit 1)
+        )
+      )

Commit message: Changes to buttons
Parts:
- SW201, SW202: symbol Switch:SW_SPST -> lzptr:TL3365AF180QG; MANUFACTURER (none) -> E-Switch; MAXIMUM_PACKAGE_HEIGHT (none) -> 2.5 mm; PARTREV (none) -> A; SNAPEDA_PN (none) -> TL3365AF180QG; STANDARD (none) -> Manufacturer Recommendations
Connections:
- net QSPI_CS: now also SW202.2
- net RUN: now also SW201.2
- net at R306.2: now also SW201.3, SW201.4; no longer SW201.2 (B)
- net at R307.2: now also SW202.3, SW202.4; no longer SW202.2 (B)
Other:
- moved on the sheet: R306, R307
