File: hardware/mcu.kicad_sch (KiCad schematic)
At the start: 44 parts, among them J201 2x5 1.27mm, J202 USB_C_Receptacle_USB2.0, SW201 RESET, SW202 BOOTSEL, U201 RP2040, U202 USBLC6-2SC6, U203 W25Q128JVS, Y201 Crystal_GND24

Commit message: Updated to kicad 8
Parts:
- renumbered R402 to R213
