File: hardware/rp2040_audioboard.kicad_pcb (KiCad board)
At the start: 4 copper layers, 65 x 75 mm, 115 parts, among them J201 2x5 1.27mm, J202 USB_C_Receptacle_USB2.0, J301 031-5640-1010, J401 031-5640-1010, U101 TLV62569DBV, U102 HT7533-1, U103 MCP6001T-E/OT, U201 STM32F103CBT6, U202 USBLC6-2SC6, U301 REF3033AIDBZT, U302 MCP6001T-E/OT, U303 ADC141S626CIMM_NOPB, U304 MCP6001T-E/OT, U401 DAC7563SDGSR, U402 MCP6001T-E/OT, Y201 16MHz

Commit message: Finished mcu schematic with the rp2040
Parts:
- removed D205: PESD3V3L1BA,115, Diode_SMD:D_SOD-323
- removed L202: CMF3216F-900-2P-T, lzptr:CMC-1206
- removed R212: 1k5, Resistor_SMD:R_0402_1005Metric
- removed R213, R214: 5k1, Resistor_SMD:R_0402_1005Metric
- added C212: 100n, Capacitor_SMD:C_0402_1005Metric, F.Cu at (179.7, 89.0)
- added C214: 100n, Capacitor_SMD:C_0402_1005Metric, F.Cu at (179.7, 91.0)
- added C215: 100n, Capacitor_SMD:C_0402_1005Metric, F.Cu at (179.7, 93.0)
- added C216: 100n, Capacitor_SMD:C_0402_1005Metric, F.Cu at (179.7, 95.0)
- added SW201: RESET, lzptr:SW_TL3365AF180QG, F.Cu at (174.8, 90.4)
- added SW202: BOOTSEL, lzptr:SW_TL3365AF180QG, F.Cu at (174.8, 95.2)
- C201: value 10u -> 30pF; footprint Capacitor_SMD:C_0603_1608Metric -> Capacitor_SMD:C_0402_1005Metric
- C202: value 10p -> 30pF
- C205: value 10p -> 1u
- C206: value 100n -> 1u
- C209: value 10n -> 100n
- C210, C211: value 1u -> 100n; footprint Capacitor_SMD:C_0603_1608Metric -> Capacitor_SMD:C_0402_1005Metric
- L201: value 10n -> CMF3216F-900-2P-T; footprint Inductor_SMD:L_0402_1005Metric -> lzptr:CMC-1206
- R201, R202: value 10k -> 27
- R203: value 0R -> 1k
- R207: value 49R9 -> 5k1
- R208: value 10k -> 5k1
- U201: value STM32F103CBT6 -> RP2040; footprint Package_QFP:LQFP-48_7x7mm_P0.5mm -> Package_DFN_QFN:QFN-56-1EP_7x7mm_P0.4mm_EP3.2x3.2mm
- Y201: value 16MHz -> Crystal_GND24
- moved R203 72.7 mm to (189.5, 75.3), turned to 0 degrees
- moved R207 69.1 mm to (189.5, 77.3)
- moved C208 68.3 mm to (186.7, 77.2), turned to 0 degrees
- moved C211 66.3 mm to (186.7, 83.1), turned to 0 degrees
- moved C210 64.7 mm to (186.7, 81.2), turned to 0 degrees
- moved R208 64.7 mm to (189.5, 79.3)
- moved C205 64.5 mm to (181.9, 77.5)
- moved C209 63.6 mm to (186.7, 79.2), turned to 0 degrees
- moved C202 63.4 mm to (181.9, 73.6), turned to 0 degrees
- moved C201 61.2 mm to (181.9, 71.6), turned to 0 degrees
- moved R202 60.9 mm to (189.5, 73.3), turned to 0 degrees
- moved C204 59.9 mm to (186.7, 71.3), turned to 0 degrees
- moved C203 58.8 mm to (181.9, 75.5), turned to 0 degrees
- moved L201 58.6 mm to (178.9, 81.3), turned to 0 degrees
- moved R201 58.3 mm to (189.5, 71.3), turned to 0 degrees
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Connections:
- C201 pad 1: +3.3V -> Net-(U201-XIN)
- C202 pad 1: /[2] MCU/HSE_IN -> Net-(C202-Pad1)
- C205 pad 1: /[2] MCU/XTAL_IN -> +3.3V
- C207 pad 1: +3.3V -> /[2] MCU/RUN
- C208 pad 1: /[2] MCU/NRST -> +3.3V
- C209 pad 1: VDDA -> +3.3V
- C210 pad 1: VDDA -> +3.3V
- C213 pad 1: VBUS -> +3.3V
- D204 pad 1: /[2] MCU/CONN_SWO -> /[2] MCU/CONN_NRST
- J201 pad 6: /[2] MCU/CONN_SWO -> unconnected-(J201-Pin_6-Pad6)
- L201 pad 1: VDDA -> /[2] MCU/USB_CMC_D-
- L201 pad 2: +3.3V -> /[2] MCU/USB_CMC_D+
- R201 pad 1: +3.3V -> /[2] MCU/USB_D+
- R201 pad 2: /[2] MCU/SPI2_NSS -> /[2] MCU/USB_DT+
- R202 pad 1: /[2] MCU/BOOT0 -> /[2] MCU/USB_D-
- R202 pad 2: GND -> /[2] MCU/USB_DT-
- R203 pad 1: /[2] MCU/HSE_OUT -> Net-(C202-Pad1)
- R203 pad 2: /[2] MCU/XTAL_IN -> Net-(U201-XOUT)
- R206 pad 1: /[2] MCU/SWO -> /[2] MCU/RUN
- R206 pad 2: /[2] MCU/CONN_SWO -> /[2] MCU/CONN_NRST
- R207 pad 1: /[2] MCU/NRST -> /[2] MCU/USB_CONN_CC1
- R207 pad 2: /[2] MCU/CONN_NRST -> GND
- R208 pad 1: +3.3V -> /[2] MCU/USB_CONN_CC2
- R208 pad 2: /[2] MCU/SPI1_NSS -> GND
- R306 pad 2: /[2] MCU/SPI1_SCK -> /[3] ADC/SPI_CLK
- R401 pad 1: /[2] MCU/SPI2_SCK -> /[4] DAC/SPI_CLK
- U201 pad 10: unconnected-(U201-PA0-Pad10) -> +3.3V
- U201 pad 14: /[2] MCU/SPI1_NSS -> unconnected-(U201-GPIO11-Pad14)
- U201 pad 15: /[2] MCU/SPI1_SCK -> unconnected-(U201-GPIO12-Pad15)
- U201 pad 16: /[2] MCU/SPI1_MISO -> unconnected-(U201-GPIO13-Pad16)
- U201 pad 19: unconnected-(U201-PB1-Pad19) -> GND
- U201 pad 20: /[2] MCU/DAC_NCLR -> Net-(U201-XIN)
- U201 pad 21: /[2] MCU/DAC_NLDAC -> Net-(U201-XOUT)
- U201 pad 22: unconnected-(U201-PB11-Pad22) -> +3.3V
- U201 pad 23: GND -> +3.3V
- U201 pad 24: +3.3V -> /[2] MCU/SWCLK
- U201 pad 25: /[2] MCU/SPI2_NSS -> /[2] MCU/SWDIO
- U201 pad 26: /[2] MCU/SPI2_SCK -> unconnected-(U201-RUN-Pad26)
- U201 pad 28: /[2] MCU/SPI2_MOSI -> unconnected-(U201-GPIO17-Pad28)
- U201 pad 32: /[2] MCU/USB_D- -> unconnected-(U201-GPIO21-Pad32)
- U201 pad 33: /[2] MCU/USB_D+ -> +3.3V
- U201 pad 34: /[2] MCU/SWDIO -> unconnected-(U201-GPIO22-Pad34)
- U201 pad 35: GND -> unconnected-(U201-GPIO23-Pad35)
- U201 pad 36: +3.3V -> unconnected-(U201-GPIO24-Pad36)
- U201 pad 37: /[2] MCU/SWCLK -> unconnected-(U201-GPIO25-Pad37)
- U201 pad 39: /[2] MCU/SWO -> unconnected-(U201-GPIO27_ADC1-Pad39)
- U201 pad 42: /[2] MCU/TIM4_CH1 -> +3.3V
- U201 pad 43: /[2] MCU/TIM4_CH2 -> +3.3V
- U201 pad 44: /[2] MCU/BOOT0 -> +3.3V
- U201 pad 45: /[2] MCU/TIM4_CH3 -> +3.3V
- U201 pad 46: unconnected-(U201-PB9-Pad46) -> /[2] MCU/USB_DT-
- U201 pad 47: GND -> /[2] MCU/USB_DT+
- U201 pad 5: /[2] MCU/HSE_IN -> unconnected-(U201-GPIO3-Pad5)
- U201 pad 6: /[2] MCU/HSE_OUT -> unconnected-(U201-GPIO4-Pad6)
- U201 pad 7: /[2] MCU/NRST -> unconnected-(U201-GPIO5-Pad7)
- U201 pad 8: GND -> unconnected-(U201-GPIO6-Pad8)
- U201 pad 9: VDDA -> unconnected-(U201-GPIO7-Pad9)
- U303 pad 6: /[2] MCU/SPI1_NSS -> /[3] ADC/SPI_ NCS
- U303 pad 7: /[2] MCU/SPI1_MISO -> /[3] ADC/SPI_MISO
- U401 pad 4: /[2] MCU/DAC_NLDAC -> /[4] DAC/DAC_NLDAC
- U401 pad 5: /[2] MCU/DAC_NCLR -> /[4] DAC/DAC_NCLR
- U401 pad 6: /[2] MCU/SPI2_NSS -> /[4] DAC/SPI_NCS
- U401 pad 8: /[2] MCU/SPI2_MOSI -> /[4] DAC/SPI_MOSI
- Y201 pad 1: /[2] MCU/HSE_IN -> Net-(U201-XIN)
- Y201 pad 3: /[2] MCU/XTAL_IN -> Net-(C202-Pad1)
Routing:
- net +3.3V: track 181.4 -> 101.8 mm, vias 13 -> 5
- net +5V: track 92.2 -> 22.6 mm, vias 4 -> 0
- net /[2] MCU/SPI2_MOSI: track 35.1 -> 0.00 mm
- net /[2] MCU/DAC_NLDAC: track 32.7 -> 0.00 mm, vias 2 -> 0
- net /[2] MCU/DAC_NCLR: track 32.5 -> 0.00 mm, vias 2 -> 0
- net /[2] MCU/SPI1_MISO: track 27.6 -> 0.00 mm
- net /[2] MCU/SPI2_NSS: track 26.4 -> 0.00 mm, vias 2 -> 0
- net GND: track 71.9 -> 49.3 mm, vias 181 -> 158
- net /[2] MCU/SPI1_NSS: track 22.3 -> 0.00 mm, vias 2 -> 0
- net /[2] MCU/SWDIO: track 20.3 -> 0.00 mm
- net /[2] MCU/SPI2_SCK: track 19.6 -> 0.00 mm
- net VBUS: track 19.0 -> 0.00 mm
- net /[2] MCU/NRST: track 18.3 -> 0.00 mm, vias 2 -> 0
- net /[2] MCU/SPI1_SCK: track 18.1 -> 0.00 mm
- net /[2] MCU/USB_D-: track 14.1 -> 0.00 mm
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- removed copper zone on F.Cu, net +5V
- removed copper zone on F.Cu, net VBUS
- removed copper zone on F.Cu, net VDDA

Commit message: Finished rp2040 schematic
Parts:
- added C217: 1u, Capacitor_SMD:C_0402_1005Metric, F.Cu at (189.9, 97.7)
- added C218: 100n, Capacitor_SMD:C_0402_1005Metric, F.Cu at (189.9, 99.7)
- added D205: Act, LED_SMD:LED_0603_1608Metric, F.Cu at (193.3, 98.0)
- added R209: 1k, Resistor_SMD:R_0402_1005Metric, F.Cu at (187.0, 91.0)
- added R210: 1k, Resistor_SMD:R_0402_1005Metric, F.Cu at (187.0, 92.9)
- added R211: 1k, Resistor_SMD:R_0402_1005Metric, F.Cu at (187.0, 94.9)
- added R212: 10k, Resistor_SMD:R_0402_1005Metric, F.Cu at (187.0, 96.9)
- added U203: W25Q128JVS, Package_SO:SOIC-8_5.23x5.23mm_P1.27mm, F.Cu at (127.0, 83.7)
- U401: value DAC7563SDGSR -> DAC7562SDGSR
- moved SW202 63.1 mm to (114.8, 75.5), turned to -90 degrees
- moved SW201 54.9 mm to (121.9, 75.5), turned to -90 degrees
- moved Y201 52.5 mm to (122.3, 92.3)
- moved U201 47.1 mm to (133.6, 96.2), turned to -90 degrees
- moved U202 38.4 mm to (155.0, 96.8)
- moved L201 32.8 mm to (149.9, 96.8)
- moved D201 24.6 mm to (106.8, 86.2), turned to 0 degrees
- moved J201 22.3 mm to (107.7, 91.2), turned to 0 degrees
- moved D202 21.9 mm to (113.3, 92.5), turned to -90 degrees
- moved D204 19.0 mm to (110.7, 96.2)
- moved C207 19.0 mm to (112.2, 97.8)
- moved R206 19.0 mm to (110.1, 97.8)
- moved R204 18.9 mm to (114.9, 92.0), turned to 90 degrees
- moved D203 15.8 mm to (113.3, 89.2), turned to -90 degrees
- moved R205 12.8 mm to (114.9, 88.5), turned to 90 degrees
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Connections:
- net Net-(U201-XIN) renamed /[2] MCU/XIN
- net Net-(U201-XOUT) renamed /[2] MCU/XOUT
- C203 pad 1: +3.3V -> +1V1
- C204 pad 1: +3.3V -> +1V1
- C205 pad 1: +3.3V -> +1V1
- C207 pad 1: /[2] MCU/RUN -> +3.3V
- C215 pad 1: +3.3V -> /[2] MCU/RUN
- R306 pad 2: /[3] ADC/SPI_CLK -> /[2] MCU/ADC_SPI1_CLK
- R401 pad 1: /[4] DAC/SPI_CLK -> /[2] MCU/DAC_SPI0_CLK
- U201 pad 2: unconnected-(U201-GPIO0-Pad2) -> /[2] MCU/ACT_LED
- U201 pad 23: +3.3V -> +1V1
- U201 pad 26: unconnected-(U201-RUN-Pad26) -> /[2] MCU/RUN
- U201 pad 29: unconnected-(U201-GPIO18-Pad29) -> /[2] MCU/ADC_SPI1_CLK
- U201 pad 31: unconnected-(U201-GPIO20-Pad31) -> /[2] MCU/ADC_SPI1_MISO
- U201 pad 32: unconnected-(U201-GPIO21-Pad32) -> /[2] MCU/ADC_SPI1_NCS
- U201 pad 34: unconnected-(U201-GPIO22-Pad34) -> /[2] MCU/DAC_SPI0_CLK
- U201 pad 35: unconnected-(U201-GPIO23-Pad35) -> /[2] MCU/DAC_SPI0_MOSI
- U201 pad 37: unconnected-(U201-GPIO25-Pad37) -> /[2] MCU/DAC_SPI0_NCS
- U201 pad 38: unconnected-(U201-GPIO26_ADC0-Pad38) -> /[2] MCU/DAC_NLDAC
- U201 pad 39: unconnected-(U201-GPIO27_ADC1-Pad39) -> /[2] MCU/DAC_NCLR
- U201 pad 45: +3.3V -> +1V1
- U201 pad 50: +3.3V -> +1V1
- U201 pad 51: unconnected-(U201-QSPI_SD3-Pad51) -> /[2] MCU/QSPI_SD3
- U201 pad 52: unconnected-(U201-QSPI_SCLK-Pad52) -> /[2] MCU/QSPI_SCLK
- U201 pad 53: unconnected-(U201-QSPI_SD0-Pad53) -> /[2] MCU/QSPI_SD0
- U201 pad 54: unconnected-(U201-QSPI_SD2-Pad54) -> /[2] MCU/QSPI_SD2
- U201 pad 55: unconnected-(U201-QSPI_SD1-Pad55) -> /[2] MCU/QSPI_SD1
- U201 pad 56: unconnected-(U201-QSPI_SS-Pad56) -> /[2] MCU/QSPI_CS
- U303 pad 6: /[3] ADC/SPI_ NCS -> /[2] MCU/ADC_SPI1_NCS
- U303 pad 7: /[3] ADC/SPI_MISO -> /[2] MCU/ADC_SPI1_MISO
- U401 pad 4: /[4] DAC/DAC_NLDAC -> /[2] MCU/DAC_NLDAC
- U401 pad 5: /[4] DAC/DAC_NCLR -> /[2] MCU/DAC_NCLR
- U401 pad 6: /[4] DAC/SPI_NCS -> /[2] MCU/DAC_SPI0_NCS
- U401 pad 8: /[4] DAC/SPI_MOSI -> /[2] MCU/DAC_SPI0_MOSI
Routing:
- net +3.3V: track 101.8 -> 45.6 mm, vias 5 -> 4
- net /[2] MCU/CONN_SWCLK: track 5.73 -> 0.00 mm
- net /[2] MCU/CONN_NRST: track 5.38 -> 0.10 mm
- net /[2] MCU/CONN_SWDIO: track 6.02 -> 1.15 mm
- net GND: track 49.3 -> 45.4 mm, vias 158 -> 128
- net /[2] MCU/RUN: track 1.11 -> 0.00 mm
- net /[3] ADC/SPI_ NCS: track 0.75 -> 0.00 mm
- net /[2] MCU/ADC_SPI1_NCS: track 0.00 -> 0.75 mm
- net +5V: track 22.6 -> 21.9 mm
Other:
- board size 65 x 75 mm -> 65.2 x 75 mm
- board text removed: "SWD"

Commit message: Finished layout changes
Parts:
- removed C218: 100n, Capacitor_SMD:C_0402_1005Metric
- C216: value 100n -> 1u
- C217: value 1u -> 100n
- moved R203 69.9 mm to (121.0, 89.0)
- moved C214 68.4 mm to (111.8, 99.0), turned to -90 degrees
- moved C204 67.7 mm to (122.3, 92.3), turned to 180 degrees
- moved C202 64.9 mm to (118.9, 89.0), turned to 180 degrees
- moved C211 64.9 mm to (122.3, 91.2), turned to 180 degrees
- moved R212 64.6 mm to (126.8, 73.5)
- moved C217 60.9 mm to (134.1, 73.2), turned to 90 degrees
- moved C201 60.7 mm to (122.7, 85.0), turned to 90 degrees
- moved C210 60.4 mm to (129.2, 99.7), turned to -90 degrees
- moved C209 56.2 mm to (134.3, 99.8), turned to -90 degrees
- moved C208 56.0 mm to (135.4, 99.8), turned to -90 degrees
- moved C213 53.9 mm to (132.8, 85.2), turned to 90 degrees
- moved L101 53.5 mm to (152.8, 95.2), turned to 180 degrees
- moved R201 53.2 mm to (140.4, 91.7), turned to 180 degrees
- moved C206 53.0 mm to (138.3, 95.0)
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Connections:
- net Net-(C202-Pad1) renamed /[2] MCU/CR_XOUT
- C214 pad 1: +3.3V -> /[2] MCU/RUN
- C215 pad 1: /[2] MCU/RUN -> VBUS
- C216 pad 1: VBUS -> +3.3V
- U201 pad 2: /[2] MCU/ACT_LED -> unconnected-(U201-GPIO0-Pad2)
- U201 pad 41: unconnected-(U201-GPIO29_ADC3-Pad41) -> /[2] MCU/ACT_LED
Routing:
- net +3.3V: track 45.6 -> 29.7 mm
- net +5V: track 21.9 -> 7.80 mm
- net /[2] MCU/USB_CONN_D+: track 3.52 -> 0.03 mm
- net GND: vias 128 -> 124
Other:
- board size 65.2 x 75 mm -> 65 x 75 mm
- board text added: "RESET"

Commit message: Finished routing
Parts:
- moved R210 59.7 mm to (116.2, 73.0), turned to 90 degrees
- moved R211 54.3 mm to (119.2, 79.0), turned to 0 degrees
- moved D205 53.8 mm to (119.5, 80.3), turned to 0 degrees
- moved SW202 53.7 mm to (113.8, 75.0), turned to 90 degrees
- moved SW201 52.4 mm to (119.8, 75.0), turned to 90 degrees
- moved R209 51.1 mm to (122.2, 73.0), turned to 90 degrees
- moved R212 12.5 mm to (134.6, 83.4), turned to 180 degrees
- moved C217 11.6 mm to (126.9, 82.2), turned to -90 degrees
- moved C216 10.4 mm to (128.0, 82.2), turned to -90 degrees
- moved R207 7.29 mm to (162.2, 98.7), turned to 180 degrees
- moved R208 6.83 mm to (162.2, 86.8), turned to 180 degrees
- moved TP102 4.04 mm to (145.3, 88.5)
- moved R204 3.48 mm to (114.9, 89.2)
- moved D202 3.47 mm to (113.3, 89.8)
- moved D203 3.35 mm to (113.3, 93.2)
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Connections:
- D202 pad 1: /[2] MCU/CONN_SWDIO -> /[2] MCU/CONN_SWCLK
- D203 pad 1: /[2] MCU/CONN_SWCLK -> /[2] MCU/CONN_SWDIO
- J201 pad 2: /[2] MCU/CONN_SWDIO -> /[2] MCU/CONN_SWCLK
- J201 pad 4: /[2] MCU/CONN_SWCLK -> /[2] MCU/CONN_SWDIO
- R204 pad 1: /[2] MCU/SWDIO -> /[2] MCU/SWCLK
- R204 pad 2: /[2] MCU/CONN_SWDIO -> /[2] MCU/CONN_SWCLK
- R205 pad 1: /[2] MCU/SWCLK -> /[2] MCU/SWDIO
- R205 pad 2: /[2] MCU/CONN_SWCLK -> /[2] MCU/CONN_SWDIO
- U201 pad 14: unconnected-(U201-GPIO11-Pad14) -> /[2] MCU/ACT_LED
- U201 pad 41: /[2] MCU/ACT_LED -> unconnected-(U201-GPIO29_ADC3-Pad41)
Routing:
- net +3.3V: track 29.7 -> 193.3 mm, vias 4 -> 13
- net +5V: track 7.80 -> 92.2 mm, vias 0 -> 4
- net /[2] MCU/RUN: track 0.00 -> 46.5 mm, vias 0 -> 2
- net /[2] MCU/DAC_NLDAC: track 0.00 -> 36.4 mm
- net /[2] MCU/DAC_NCLR: track 0.00 -> 36.4 mm
- net /[2] MCU/QSPI_SD3: track 0.00 -> 36.0 mm
- net /[2] MCU/DAC_SPI0_MOSI: track 0.00 -> 35.9 mm
- net /[2] MCU/QSPI_CS: track 0.00 -> 33.7 mm, vias 0 -> 2
- net /[2] MCU/QSPI_SCLK: track 0.00 -> 32.2 mm
- net /[2] MCU/DAC_SPI0_NCS: track 0.00 -> 29.0 mm, vias 0 -> 2
- net /[2] MCU/QSPI_SD0: track 0.00 -> 26.8 mm
- net +1V1: track 0.00 -> 25.9 mm
- net /[2] MCU/DAC_SPI0_CLK: track 0.00 -> 24.6 mm
- net GND: track 45.4 -> 69.0 mm, vias 124 -> 173
- net VBUS: track 0.00 -> 23.1 mm
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- added copper zone on B.Cu, net +3.3V
Other:
- board text added: "BOOTSEL"
- board text added: "JLCJLCJLCJLC"
- board text added: "LP 05/23 REV A"
- board text removed: "LP 03/23 REV A"
- board text removed: "USB"

Commit message: Finished bom
Parts:
- R212: value 10k -> DNP 10k
- U103, U302, U304, U402: value MCP6001T-E/OT -> TLV9001IDBVR
Connections:
- D202 pad 1: /[2] MCU/CONN_SWCLK -> /[2] MCU/CONN_SWDIO
- D203 pad 1: /[2] MCU/CONN_SWDIO -> /[2] MCU/CONN_SWCLK
- J201 pad 2: /[2] MCU/CONN_SWCLK -> /[2] MCU/CONN_SWDIO
- J201 pad 4: /[2] MCU/CONN_SWDIO -> /[2] MCU/CONN_SWCLK
- R204 pad 1: /[2] MCU/SWCLK -> /[2] MCU/SWDIO
- R204 pad 2: /[2] MCU/CONN_SWCLK -> /[2] MCU/CONN_SWDIO
- R205 pad 1: /[2] MCU/SWDIO -> /[2] MCU/SWCLK
- R205 pad 2: /[2] MCU/CONN_SWDIO -> /[2] MCU/CONN_SWCLK
Routing:
- net /[2] MCU/SWDIO: track 12.8 -> 18.3 mm, vias 0 -> 2
- net /[2] MCU/SWCLK: track 13.8 -> 12.3 mm
- net /[2] MCU/CONN_SWDIO: track 6.48 -> 5.43 mm
- net /[2] MCU/CONN_SWCLK: track 5.43 -> 6.48 mm

Commit message: Cleanup, minor bom changes and finished production files
Parts:
- D201, D202, D203, D204, D301, D401: value PESD3V3L1BA,115 -> PESD3V3L1BA
Routing:
- net GND: vias 173 -> 175
Changed lines of the file:
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@@
     (tags "SOD-323")
     (property "LCSC Part #" "")
-    (property "MPN" "C51450")
-    (property "Rating" "5.8V 26V")
+    (property "MPN" "C2939000")
+    (property "Rating" "4V 10.5V")
     (property "Sheetfile" "mcu.kicad_sch")
     (property "Sheetname" "[2] MCU")
@@
         (effects (font (size 1 1) (thickness 0.15)))
     )
-    (fp_text value "PESD3V3L1BA,115" (at 0.1 1.9 90) (layer "F.Fab")
+    (fp_text value "PESD3V3L1BA" (at 0.1 1.9 90) (layer "F.Fab")
         (effects (font (size 1 1) (thickness 0.15)))
     )
@@
     (descr "SOIC, 8 Pin (http://www.winbond.com/resource-files/w25q32jv%20revg%2003272018%20plus.pdf#page=68), generated with kicad-footprint-generator ipc_gullwing_generator.py")
     (tags "SOIC SO")
-    (property "MPN" "C113767")
+    (property "MPN" "C97521")
     (property "Rating" "")
     (property "Sheetfile" "mcu.kicad_sch")
@@
     (tags "SOD-323")
     (property "LCSC Part #" "")
-    (property "MPN" "C51450")
-    (property "Rating" "5.8V 26V")
+    (property "MPN" "C2939000")
+    (property "Rating" "4V 10.5V")
     (property "Sheetfile" "mcu.kicad_sch")
     (property "Sheetname" "[2] MCU")
@@
         (effects (font (size 1 1) (thickness 0.15)))
     )
-    (fp_text value "PESD3V3L1BA,115" (at 0.1 1.9) (layer "F.Fab")
+    (fp_text value "PESD3V3L1BA" (at 0.1 1.9) (layer "F.Fab")
         (effects (font (size 1 1) (thickness 0.15)))
     )
@@
     (descr "LED SMD 0603 (1608 Metric), square (rectangular) end terminal, IPC_7351 nominal, (Body size source: http://www.tortai-tech.com/upload/download/2011102023233369053.pdf), generated with kicad-footprint-generator")
     (tags "LED")
-    (property "MPN" "C2292")
+    (property "MPN" "C72043")
     (property "Rating" "Green")
     (property "Sheetfile" "mcu.kicad_sch")
@@
     (tags "SOD-323")
     (property "LCSC Part #" "")
-    (property "MPN" "C51450")
-    (property "Rating" "5.8V 26V")
+    (property "MPN" "C2939000")
+    (property "Rating" "4V 10.5V")
     (property "Sheetfile" "dac.kicad_sch")
     (property "Sheetname" "[4] DAC")
@@
         (effects (font (size 1 1) (thickness 0.15)))
     )
-    (fp_text value "PESD3V3L1BA,115" (at 0.1 1.9) (layer "F.Fab")
+    (fp_text value "PESD3V3L1BA" (at 0.1 1.9) (layer "F.Fab")
         (effects (font (size 1 1) (thickness 0.15)))
     )
@@
     (descr "Inductor SMD 0402 (1005 Metric), square (rectangular) end terminal, IPC_7351 nominal, (Body size source: http://www.tortai-tech.com/upload/download/2011102023233369053.pdf), generated with kicad-footprint-generator")
     (tags "inductor")
-    (property "MPN" "C961338")
+    (property "MPN" "C361500")
     (property "Rating" "")
     (property "Sheetfile" "power.kicad_sch")
@@
     (tags "SOD-323")
     (property "LCSC Part #" "")
-    (property "MPN" "C51450")
-    (property "Rating" "5.8V 26V")
+    (property "MPN" "C2939000")
+    (property "Rating" "4V 10.5V")
     (property "Sheetfile" "mcu.kicad_sch")
     (property "Sheetname" "[2] MCU")
@@
         (effects (font (size 1 1) (thickness 0.15)))
     )
-    (fp_text value "PESD3V3L1BA,115" (at 0.1 1.9 90) (layer "F.Fab")
+    (fp_text value "PESD3V3L1BA" (at 0.1 1.9 90) (layer "F.Fab")
         (effects (font (size 1 1) (thickness 0.15)))
     )
@@
     (descr "LED SMD 0603 (1608 Metric), square (rectangular) end terminal, IPC_7351 nominal, (Body size source: http://www.tortai-tech.com/upload/download/2011102023233369053.pdf), generated with kicad-footprint-generator")
     (tags "LED")
-    (property "MPN" "C2292")
+    (property "MPN" "C72043")
     (property "Rating" "Green")
     (property "Sheetfile" "power.kicad_sch")
@@
     (tags "SOD-323")
     (property "LCSC Part #" "")
-    (property "MPN" "C51450")
-    (property "Rating" "5.8V 26V")
+    (property "MPN" "C2939000")
+    (property "Rating" "4V 10.5V")
     (property "Sheetfile" "mcu.kicad_sch")
     (property "Sheetname" "[2] MCU")
@@
         (effects (font (size 1 1) (thickness 0.15)))
     )
-    (fp_text value "PESD3V3L1BA,115" (at 0.1 1.9) (layer "F.Fab")
+    (fp_text value "PESD3V3L1BA" (at 0.1 1.9) (layer "F.Fab")
         (effects (font (size 1 1) (thickness 0.15)))
     )
@@
     (descr "LED SMD 0603 (1608 Metric), square (rectangular) end terminal, IPC_7351 nominal, (Body size source: http://www.tortai-tech.com/upload/download/2011102023233369053.pdf), generated with kicad-footprint-generator")
     (tags "LED")
-    (property "MPN" "C2292")
+    (property "MPN" "C72043")
     (property "Rating" "Green")
     (property "Sheetfile" "power.kicad_sch")
@@
   )
   (footprint "Resistor_SMD:R_0402_1005Metric" (layer "F.Cu")
-    (at 116.15 72.95 90)
+    (at 116.2 72.95 90)
     (descr "Resistor SMD 0402 (1005 Metric), square (rectangular) end terminal, IPC_7351 nominal, (Body size source: IPC-SM-782 page 72, https://www.pcb-3d.com/wordpress/wp-content/uploads/ipc-sm-782a_amendment_1_and_2.pdf), generated with kicad-footprint-generator")
     (tags "resistor")
@@
     (tags "SOD-323")
     (property "LCSC Part #" "")
-    (property "MPN" "C51450")
-    (property "Rating" "5.8V 26V")
+    (property "MPN" "C2939000")
+    (property "Rating" "4V 10.5V")
     (property "Sheetfile" "adc.kicad_sch")
     (property "Sheetname" "[3] ADC")
@@
         (effects (font (size 1 1) (thickness 0.15)))
     )
-    (fp_text value "PESD3V3L1BA,115" (at 0.1 1.9) (layer "F.Fab")
+    (fp_text value "PESD3V3L1BA" (at 0.1 1.9) (layer "F.Fab")
         (effects (font (size 1 1) (thickness 0.15)))
     )
@@
   (gr_line (start 166.5 140.75) (end 166.5 75.75)
     (stroke (width 0.0381) (type default)) (layer "Edge.Cuts"))
-  (gr_text "LP 05/23\nREV A" (at 131.2 141.35) (layer "F.SilkS")
+  (gr_text "LP 05/23\nREV A" (at 130.6 141.35) (layer "F.SilkS")
     (effects (font (size 1 1) (thickness 0.2)) (justify left bottom))
   )
-  (gr_text "BOOTSEL" (at 111.8 78.05 90) (layer "F.SilkS")
+  (gr_text "BOOTSEL" (at 111.8 77.65 90) (layer "F.SilkS")
     (effects (font (size 0.8 0.8) (thickness 0.15) bold) (justify left bottom))
   )
@@
     (effects (font (size 0.8 0.8) (thickness 0.15)))
   )
-  (gr_text "RESET" (at 122.85 78.1 90) (layer "F.SilkS")
+  (gr_text "RESET" (at 117.9 77.65 90) (layer "F.SilkS")
     (effects (font (size 0.8 0.8) (thickness 0.15) bold) (justify left bottom))
   )
@@
   (via (at 164 128.25) (size 0.8) (drill 0.4) (layers "F.Cu" "B.Cu") (free) (net 2))
   (via (at 152.1 119.55) (size 0.7) (drill 0.3) (layers "F.Cu" "B.Cu") (net 2))
+  (via (at 104 113.15) (size 0.8) (drill 0.4) (layers "F.Cu" "B.Cu") (free) (net 2))
   (via (at 129 92.25) (size 0.7) (drill 0.3) (layers "F.Cu" "B.Cu") (net 2))
   (via (at 164 117.95) (size 0.8) (drill 0.4) (layers "F.Cu" "B.Cu") (free) (net 2))
   (via (at 129 143.25) (size 0.8) (drill 0.4) (layers "F.Cu" "B.Cu") (free) (net 2))
   (via (at 148.9 114.75) (size 0.7) (drill 0.3) (layers "F.Cu" "B.Cu") (net 2))
+  (via (at 104 108.05) (size 0.8) (drill 0.4) (layers "F.Cu" "B.Cu") (free) (net 2))
   (via (at 124 113.25) (size 0.8) (drill 0.4) (layers "F.Cu" "B.Cu") (free) (net 2))
   (via (at 131.5 108.25) (size 0.8) (drill 0.4) (layers "F.Cu" "B.Cu") (free) (net 2))
@@
   (segment (start 122.25 72.44) (end 121.91 72.44) (width 0.3) (layer "F.Cu") (net 52))
   (segment (start 121.91 72.44) (end 121.6 72.75) (width 0.3) (layer "F.Cu") (net 52))
-  (segment (start 116.01 72.44) (end 115.7 72.75) (width 0.3) (layer "F.Cu") (net 53))
-  (segment (start 115.7 72.75) (end 114.825 72.75) (width 0.3) (layer "F.Cu") (net 53))
-  (segment (start 116.15 72.44) (end 116.01 72.44) (width 0.3) (layer "F.Cu") (net 53))
+  (segment (start 115.89 72.75) (end 116.2 72.44) (width 0.3) (layer "F.Cu") (net 53))
+  (segment (start 114.825 72.75) (end 115.89 72.75) (width 0.3) (layer "F.Cu") (net 53))
   (segment (start 126.5 124.45) (end 124.01 124.45) (width 0.3) (layer "F.Cu") (net 54))
   (segment (start 134.5 123.15) (end 134.5 121.75) (width 0.3) (layer "F.Cu") (net 54))
