File: hardware/rp2040_audioboard.kicad_pcb (KiCad board)
At the start: 4 copper layers, 65 x 75 mm, 123 parts, among them J201 2x5 1.27mm, J202 USB_C_Receptacle_USB2.0, J301 031-5640-1010, J401 031-5640-1010, SW201 RESET, SW202 BOOTSEL, U101 TLV62569DBV, U102 HT7533-1, U103 TLV9001IDBVR, U201 RP2040, U202 USBLC6-2SC6, U203 W25Q128JVS, U301 REF3033AIDBZT, U302 TLV9001IDBVR, U303 ADC141S626CIMM_NOPB, U304 TLV9001IDBVR, U401 DAC7562SDGSR, U402 TLV9001IDBVR, Y201 Crystal_GND24

Commit message: Fixed missing pull up for run pin
Parts:
- added R213: 10k, Resistor_SMD:R_0402_1005Metric, F.Cu at (124.1, 95.8)
Routing:
- net +3.3V: track 193.3 -> 194.5 mm, vias 13 -> 14
- net /[2] MCU/RUN: track 46.5 -> 47.4 mm
Other:
- board text added: "LP 07/23 REV B"
- board text removed: "LP 05/23 REV A"
Changed lines of the file:
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@@
     )
   )
+  (footprint "Resistor_SMD:R_0402_1005Metric" (layer "F.Cu")
+    (at 124.1 95.85 180)
+    (descr "Resistor SMD 0402 (1005 Metric), square (rectangular) end terminal, IPC_7351 nominal, (Body size source: IPC-SM-782 page 72, https://www.pcb-3d.com/wordpress/wp-content/uploads/ipc-sm-782a_amendment_1_and_2.pdf), generated with kicad-footprint-generator")
+    (tags "resistor")
+    (property "MPN" "C25744")
+    (property "Rating" "63mW")
+    (property "Sheetfile" "mcu.kicad_sch")
+    (property "Sheetname" "[2] MCU")
+    (property "ki_description" "Resistor")
+    (property "ki_keywords" "R res resistor")
+    (attr smd)
+    (fp_text reference "R213" (at 0 -1.17) (layer "F.SilkS") hide
+        (effects (font (size 1 1) (thickness 0.15)))
+    )
+    (fp_text value "10k" (at 0 1.17) (layer "F.Fab")
+        (effects (font (size 1 1) (thickness 0.15)))
+    )
+    (fp_text user "${REFERENCE}" (at 0 0) (layer "F.Fab")
+        (effects (font (size 0.26 0.26) (thickness 0.04)))
+    )
+    (fp_line (start -0.153641 -0.38) (end 0.153641 -0.38)
+      (stroke (width 0.12) (type solid)) (layer "F.SilkS"))
+    (fp_line (start -0.153641 0.38) (end 0.153641 0.38)
+      (stroke (width 0.12) (type solid)) (layer "F.SilkS"))
+    (fp_line (start -0.93 -0.47) (end 0.93 -0.47)
+      (stroke (width 0.05) (type solid)) (layer "F.CrtYd"))
+    (fp_line (start -0.93 0.47) (end -0.93 -0.47)
+      (stroke (width 0.05) (type solid)) (layer "F.CrtYd"))
+    (fp_line (start 0.93 -0.47) (end 0.93 0.47)
+      (stroke (width 0.05) (type solid)) (layer "F.CrtYd"))
+    (fp_line (start 0.93 0.47) (end -0.93 0.47)
+      (stroke (width 0.05) (type solid)) (layer "F.CrtYd"))
+    (fp_line (start -0.525 -0.27) (end 0.525 -0.27)
+      (stroke (width 0.1) (type solid)) (layer "F.Fab"))
+    (fp_line (start -0.525 0.27) (end -0.525 -0.27)
+      (stroke (width 0.1) (type solid)) (layer "F.Fab"))
+    (fp_line (start 0.525 -0.27) (end 0.525 0.27)
+      (stroke (width 0.1) (type solid)) (layer "F.Fab"))
+    (fp_line (start 0.525 0.27) (end -0.525 0.27)
+      (stroke (width 0.1) (type solid)) (layer "F.Fab"))
+    (pad "1" smd roundrect (at -0.51 0 180) (size 0.54 0.64) (layers "F.Cu" "F.Paste" "F.Mask") (roundrect_rratio 0.25)
+      (net 4 "+3.3V") (pintype "passive"))
+    (pad "2" smd roundrect (at 0.51 0 180) (size 0.54 0.64) (layers "F.Cu" "F.Paste" "F.Mask") (roundrect_rratio 0.25)
+      (net 9 "/[2] MCU/RUN") (pintype "passive"))
+    (model "${KICAD6_3DMODEL_DIR}/Resistor_SMD.3dshapes/R_0402_1005Metric.wrl"
+      (offset (xyz 0 0 0))
+      (scale (xyz 1 1 1))
+      (rotate (xyz 0 0 0))
+    )
+  )
   (footprint "Capacitor_SMD:C_0402_1005Metric" (layer "F.Cu")
     (at 114.55 114.85)
@@
     (property "Sheetfile" "mcu.kicad_sch")
     (property "Sheetname" "[2] MCU")
-    (property "ki_description" "Resistor, US symbol")
+    (property "ki_description" "Resistor")
     (property "ki_keywords" "R res resistor")
     (property "mpn" "")
@@
     (property "Sheetfile" "mcu.kicad_sch")
     (property "Sheetname" "[2] MCU")
-    (property "ki_description" "Resistor, US symbol")
+    (property "ki_description" "Resistor")
     (property "ki_keywords" "R res resistor")
     (property "mpn" "")
@@
     (property "Sheetfile" "mcu.kicad_sch")
     (property "Sheetname" "[2] MCU")
-    (property "ki_description" "Resistor, US symbol")
+    (property "ki_description" "Resistor")
     (property "ki_keywords" "R res resistor")
     (property "mpn" "")
@@
   (gr_line (start 166.5 140.75) (end 166.5 75.75)
     (stroke (width 0.0381) (type default)) (layer "Edge.Cuts"))
-  (gr_text "LP 05/23\nREV A" (at 130.6 141.35) (layer "F.SilkS")
+  (gr_text "LP 07/23\nREV B" (at 130.6 141.35) (layer "F.SilkS")
     (effects (font (size 1 1) (thickness 0.2)) (justify left bottom))
   )
@@
   (segment (start 134.04 84.574386) (end 132.984386 85.63) (width 0.5) (layer "F.Cu") (net 4))
   (segment (start 146.25 103.3) (end 146.25 104.725) (width 0.3) (layer "F.Cu") (net 4))
+  (segment (start 124.61 95.85) (end 125.4 95.85) (width 0.5) (layer "F.Cu") (net 4))
   (segment (start 132.8 87.6125) (end 132.8 85.63) (width 0.2) (layer "F.Cu") (net 4))
   (segment (start 103.9 82.85) (end 103.1 83.65) (width 0.5) (layer "F.Cu") (net 4))
@@
   (via (at 129.2 86.55) (size 0.7) (drill 0.3) (layers "F.Cu" "B.Cu") (free) (net 4))
   (via (at 134.6 95.3) (size 0.7) (drill 0.3) (layers "F.Cu" "B.Cu") (free) (net 4))
+  (via (at 125.4 95.85) (size 0.7) (drill 0.3) (layers "F.Cu" "B.Cu") (net 4))
   (via (at 124.2 91.25) (size 0.7) (drill 0.3) (layers "F.Cu" "B.Cu") (free) (net 4))
   (via (at 133.9 94.7) (size 0.7) (drill 0.3) (layers "F.Cu" "B.Cu") (free) (net 4))
@@
   (segment (start 154.8 84.75) (end 154.8 80.95) (width 0.29337) (layer "B.Cu") (net 4))
   (segment (start 154.4 80.55) (end 153.2 79.35) (width 0.5) (layer "B.Cu") (net 4))
+  (segment (start 125.4 95.85) (end 125 95.85) (width 0.5) (layer "B.Cu") (net 4))
   (segment (start 150.1 85.15) (end 154.4 85.15) (width 0.29337) (layer "B.Cu") (net 4))
   (segment (start 148.24 85.09) (end 148.27 85.12) (width 0.29337) (layer "F.Cu") (net 5))
@@
   (segment (start 133.3625 123.45) (end 133.3625 123.9125) (width 0.3) (layer "F.Cu") (net 8))
   (segment (start 120.825 76.525) (end 120.35 76.05) (width 0.2) (layer "F.Cu") (net 9))
-  (segment (start 119.877058 98.57) (end 117.35 98.57) (width 0.2) (layer "F.Cu") (net 9))
   (segment (start 117.15 76.05) (end 116.7 76.5) (width 0.2) (layer "F.Cu") (net 9))
-  (segment (start 126.7625 92.85) (end 125.597058 92.85) (width 0.2) (layer "F.Cu") (net 9))
   (segment (start 116.45 76.75) (end 116.45 80.7) (width 0.2) (layer "F.Cu") (net 9))
   (segment (start 116.7 76.5) (end 116.45 76.75) (width 0.2) (layer "F.Cu") (net 9))
   (segment (start 120.825 77.25) (end 120.825 76.525) (width 0.2) (layer "F.Cu") (net 9))
   (segment (start 117.35 98.57) (end 111.8 98.57) (width 0.2) (layer "F.Cu") (net 9))
+  (segment (start 123.6 96.65) (end 123.59 96.64) (width 0.2) (layer "F.Cu") (net 9))
+  (segment (start 121.68 98.57) (end 123.6 96.65) (width 0.2) (layer "F.Cu") (net 9))
+  (segment (start 123.59 95.16) (end 125.9 92.85) (width 0.2) (layer "F.Cu") (net 9))
   (segment (start 110.63 98.57) (end 110.61 98.55) (width 0.29337) (layer "F.Cu") (net 9))
   (segment (start 116.45 97.35) (end 116.45 98) (width 0.2) (layer "F.Cu") (net 9))
   (segment (start 116.45 98) (end 117.02 98.57) (width 0.2) (layer "F.Cu") (net 9))
+  (segment (start 117.35 98.57) (end 121.68 98.57) (width 0.2) (layer "F.Cu") (net 9))
+  (segment (start 123.59 96.64) (end 123.59 95.85) (width 0.2) (layer "F.Cu") (net 9))
   (segment (start 111.8 98.57) (end 110.63 98.57) (width 0.29337) (layer "F.Cu") (net 9))
+  (segment (start 125.9 92.85) (end 126.7625 92.85) (width 0.2) (layer "F.Cu") (net 9))
+  (segment (start 123.59 95.85) (end 123.59 95.16) (width 0.2) (layer "F.Cu") (net 9))
   (segment (start 120.35 76.05) (end 117.15 76.05) (width 0.2) (layer "F.Cu") (net 9))
   (segment (start 117.02 98.57) (end 117.35 98.57) (width 0.2) (layer "F.Cu") (net 9))
-  (segment (start 125.597058 92.85) (end 119.877058 98.57) (width 0.2) (layer "F.Cu") (net 9))
   (via (at 116.45 97.35) (size 0.7) (drill 0.3) (layers "F.Cu" "B.Cu") (net 9))
   (via (at 116.45 80.7) (size 0.7) (drill 0.3) (layers "F.Cu" "B.Cu") (net 9))

Commit message: Changes to buttons
Parts:
- turned SW201 to -90 degrees
- turned SW202 to -90 degrees
Connections:
- R209 pad 2: Net-(SW201-B) -> Net-(R209-Pad2)
- R210 pad 2: Net-(SW202-B) -> Net-(R210-Pad2)
- SW201 pad 2: Net-(SW201-B) -> /[2] MCU/RUN
- SW201 pad 3: (no net) -> Net-(R209-Pad2)
- SW201 pad 4: (no net) -> Net-(R209-Pad2)
- SW202 pad 2: Net-(SW202-B) -> /[2] MCU/QSPI_CS
- SW202 pad 3: (no net) -> Net-(R210-Pad2)
- SW202 pad 4: (no net) -> Net-(R210-Pad2)
Routing:
- net Net-(R209-Pad2): track 0.00 -> 6.05 mm
- net Net-(R210-Pad2): track 0.00 -> 6.00 mm
- net /[2] MCU/QSPI_CS: track 33.7 -> 38.4 mm
- net Net-(SW201-B): track 1.55 -> 0.00 mm
- net Net-(SW202-B): track 1.50 -> 0.00 mm
- net /[2] MCU/RUN: track 47.4 -> 46.7 mm
