File: hardware/adc.kicad_sch (KiCad schematic)
At the start: 32 parts, among them J301 031-5640-1010, U301 REF3033AIDBZT, U302 MCP6001T-E/OT, U303 ADC141S626CIMM_NOPB, U304 MCP6001T-E/OT

Commit message: Finished mcu schematic with the rp2040
Parts:
- U303: MPN ADC141S626CIMM/NOPB -> C206494
Changed lines of the file:
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@@
       (effects (font (size 1.27 1.27)))
     )
-    (property "MPN" "ADC141S626CIMM/NOPB" (at 116.84 127 0)
+    (property "MPN" "C206494" (at 116.84 127 0)
       (effects (font (size 1.27 1.27)))
     )

Commit message: Finished routing
Parts:
- C304, C307, C308, C309, C310, C315: MPN CC0402KRX5R6BB104 -> C1525; Rating 10V -> 16V
Changed lines of the file:
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@@
       (effects (font (size 1.27 1.27)) hide)
     )
-    (property "MPN" "CC0402KRX5R6BB104" (at 71.12 46.99 0)
-      (effects (font (size 1.27 1.27)) hide)
-    )
-    (property "Rating" "10V" (at 71.12 41.91 90)
+    (property "MPN" "C1525" (at 71.12 46.99 0)
+      (effects (font (size 1.27 1.27)) hide)
+    )
+    (property "Rating" "16V" (at 71.12 41.91 90)
       (effects (font (size 1.27 1.27)))
     )
@@
   )
   (symbol (lib_id "Device:C") (at 134.62 102.87 0) (unit 1)
-    (in_bom yes) (on_board yes) (dnp no) (fields_autoplaced)
-    (property "Reference" "C310" (at 138.43 101.5999 0)
-      (effects (font (size 1.27 1.27)) (justify left))
-    )
-    (property "Value" "100n" (at 138.43 104.1399 0)
+    (in_bom yes) (on_board yes) (dnp no)
+    (property "Reference" "C310" (at 137.16 101.6 0)
+      (effects (font (size 1.27 1.27)) (justify left))
+    )
+    (property "Value" "100n" (at 137.16 104.14 0)
       (effects (font (size 1.27 1.27)) (justify left))
     )
@@
       (effects (font (size 1.27 1.27)) hide)
     )
-    (property "MPN" "CC0402KRX5R6BB104" (at 134.62 102.87 0)
-      (effects (font (size 1.27 1.27)) hide)
-    )
-    (property "Rating" "10V" (at 134.62 102.87 0)
-      (effects (font (size 1.27 1.27)) hide)
+    (property "MPN" "C1525" (at 134.62 102.87 0)
+      (effects (font (size 1.27 1.27)) hide)
+    )
+    (property "Rating" "16V" (at 137.16 106.6801 0)
+      (effects (font (size 1.27 1.27)) (justify left))
     )
     (pin "1")
@@
       (effects (font (size 1.27 1.27)) hide)
     )
-    (property "MPN" "CC0402KRX5R6BB104" (at 99.06 39.37 0)
-      (effects (font (size 1.27 1.27)) hide)
-    )
-    (property "Rating" "10V" (at 99.06 39.37 0)
+    (property "MPN" "C1525" (at 99.06 39.37 0)
+      (effects (font (size 1.27 1.27)) hide)
+    )
+    (property "Rating" "16V" (at 99.06 39.37 0)
       (effects (font (size 1.27 1.27)) hide)
     )
@@
   )
   (symbol (lib_id "Device:C") (at 96.52 102.87 0) (mirror y) (unit 1)
-    (in_bom yes) (on_board yes) (dnp no) (fields_autoplaced)
-    (property "Reference" "C307" (at 92.71 101.5999 0)
-      (effects (font (size 1.27 1.27)) (justify left))
-    )
-    (property "Value" "100n" (at 92.71 104.1399 0)
+    (in_bom yes) (on_board yes) (dnp no)
+    (property "Reference" "C307" (at 93.98 101.6 0)
+      (effects (font (size 1.27 1.27)) (justify left))
+    )
+    (property "Value" "100n" (at 93.98 104.14 0)
       (effects (font (size 1.27 1.27)) (justify left))
     )
@@
       (effects (font (size 1.27 1.27)) hide)
     )
-    (property "MPN" "CC0402KRX5R6BB104" (at 96.52 102.87 0)
-      (effects (font (size 1.27 1.27)) hide)
-    )
-    (property "Rating" "10V" (at 96.52 102.87 0)
-      (effects (font (size 1.27 1.27)) hide)
+    (property "MPN" "C1525" (at 96.52 102.87 0)
+      (effects (font (size 1.27 1.27)) hide)
+    )
+    (property "Rating" "16V" (at 92.71 106.6801 0)
+      (effects (font (size 1.27 1.27)) (justify left))
     )
     (pin "1")
@@
     (property "Rating" "125mW" (at 36.83 127 90)
       (effects (font (size 1.27 1.27)))
+    )
+    (property "MPN" "" (at 36.83 121.92 0)
+      (effects (font (size 1.27 1.27)) hide)
     )
     (pin "1")
@@
   )
   (symbol (lib_id "Device:C") (at 96.52 139.7 0) (mirror y) (unit 1)
-    (in_bom yes) (on_board yes) (dnp no) (fields_autoplaced)
-    (property "Reference" "C308" (at 92.71 138.4299 0)
-      (effects (font (size 1.27 1.27)) (justify left))
-    )
-    (property "Value" "100n" (at 92.71 140.9699 0)
+    (in_bom yes) (on_board yes) (dnp no)
+    (property "Reference" "C308" (at 93.98 138.43 0)
+      (effects (font (size 1.27 1.27)) (justify left))
+    )
+    (property "Value" "100n" (at 93.98 140.97 0)
       (effects (font (size 1.27 1.27)) (justify left))
     )
@@
       (effects (font (size 1.27 1.27)) hide)
     )
-    (property "MPN" "CC0402KRX5R6BB104" (at 96.52 139.7 0)
-      (effects (font (size 1.27 1.27)) hide)
-    )
-    (property "Rating" "10V" (at 96.52 139.7 0)
-      (effects (font (size 1.27 1.27)) hide)
+    (property "MPN" "C1525" (at 96.52 139.7 0)
+      (effects (font (size 1.27 1.27)) hide)
+    )
+    (property "Rating" "16V" (at 92.71 143.5101 0)
+      (effects (font (size 1.27 1.27)) (justify left))
     )
     (pin "1")
@@
       (effects (font (size 1.27 1.27)) hide)
     )
-    (property "MPN" "CC0402KRX5R6BB104" (at 181.61 41.91 0)
-      (effects (font (size 1.27 1.27)) hide)
-    )
-    (property "Rating" "10V" (at 185.42 40.64 90)
-      (effects (font (size 1.27 1.27)))
-    )
+    (property "MPN" "C1525" (at 181.61 41.91 0)
+      (effects (font (size 1.27 1.27)) hide)
+    )
+    (property "Rating" "16V" (at 185.42 40.64 90)
+      (effects (font (size 1.27 1.27)))
+    )

Commit message: Finished bom
Parts:
- C301, C302, C305, C306, C312: MPN (none) -> C96446; Rating (none) -> 25V
- C303, C314, C316: MPN (none) -> C1527; Rating (none) -> 50V
- C311, C313: MPN (none) -> C1523; Rating (none) -> 50V
- D301: MPN (none) -> C51450; Rating (none) -> 5.8V 26V
- R301: MPN (none) -> C17720
- R302, R309, R310: MPN (none) -> C11702
- R303, R304: MPN (none) -> C174169
- R305: MPN (none) -> C25917
- R306: MPN (none) -> C17168
- R307: MPN (none) -> C25768
- R308: MPN (none) -> C25752
- U301: MPN (none) -> C2872391
- U302, U304: value MCP6001T-E/OT -> TLV9001IDBVR; MPN (none) -> C398363
Changed lines of the file:
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@@
+    (stroke (width 0) (type default))
+  )
+  (wire (pts (xy 81.28 46.99) (xy 104.14 46.99))
     (stroke (width 0) (type default))
   )
@@
   )
   (wire (pts (xy 104.14 52.07) (xy 101.6 52.07))
-    (stroke (width 0) (type default))
-  )
-  (wire (pts (xy 81.28 46.99) (xy 104.14 46.99))
     (stroke (width 0) (type default))
   )
@@
     (effects (font (size 1.27 1.27)) (justify right bottom))
   )
-  (label "IN_BUF" (at 92.71 46.99 180) (fields_autoplaced)
+  (label "IN_BUF" (at 99.06 46.99 180) (fields_autoplaced)
     (effects (font (size 1.27 1.27)) (justify right bottom))
   )
@@
       (effects (font (size 1.27 1.27)) hide)
     )
+    (property "MPN" "C96446" (at 44.45 134.62 0)
+      (effects (font (size 1.27 1.27)) hide)
+    )
+    (property "Rating" "25V" (at 44.45 134.62 0)
+      (effects (font (size 1.27 1.27)) hide)
+    )
     (pin "1")
     (pin "2")
@@
       (effects (font (size 1.27 1.27)))
     )
+    (property "MPN" "C17168" (at 147.32 123.19 0)
+      (effects (font (size 1.27 1.27)) hide)
+    )
     (pin "1")
     (pin "2")
@@
     )
     (property "LCSC Part #" "" (at 39.37 53.34 90)
+      (effects (font (size 1.27 1.27)) hide)
+    )
+    (property "MPN" "C51450" (at 39.37 53.34 0)
+      (effects (font (size 1.27 1.27)) hide)
+    )
+    (property "Rating" "5.8V 26V" (at 39.37 53.34 0)
       (effects (font (size 1.27 1.27)) hide)
     )
@@
       (effects (font (size 1.27 1.27)) hide)
     )
+    (property "MPN" "C96446" (at 29.21 134.62 0)
+      (effects (font (size 1.27 1.27)) hide)
+    )
+    (property "Rating" "25V" (at 29.21 134.62 0)
+      (effects (font (size 1.27 1.27)) hide)
+    )
     (pin "1")
     (pin "2")
@@
       (effects (font (size 1.27 1.27)) (justify left))
     )
-    (property "Value" "MCP6001T-E/OT" (at 110.49 54.61 0)
+    (property "Value" "TLV9001IDBVR" (at 110.49 54.61 0)
       (effects (font (size 1.27 1.27)) (justify left))
     )
@@
       (effects (font (size 1.27 1.27)) (justify left) hide)
     )
-    (property "Datasheet" "http://ww1.microchip.com/downloads/en/DeviceDoc/21733j.pdf" (at 111.76 44.45 0)
+    (property "Datasheet" "https://www.ti.com/lit/ds/symlink/tlv9001.pdf?ts=1684276162908&ref_url=https%253A%252F%252Fwww.ti.com%252Fproduct%252FTLV9001" (at 111.76 44.45 0)
+      (effects (font (size 1.27 1.27)) hide)
+    )
+    (property "MPN" "C398363" (at 111.76 49.53 0)
       (effects (font (size 1.27 1.27)) hide)
     )
@@
       (effects (font (size 1.27 1.27)) hide)
     )
+    (property "MPN" "C1527" (at 166.37 55.88 0)
+      (effects (font (size 1.27 1.27)) hide)
+    )
+    (property "Rating" "50V" (at 166.37 55.88 0)
+      (effects (font (size 1.27 1.27)) hide)
+    )
     (pin "1")
     (pin "2")
@@
     (property "Datasheet" "http://www.ti.com/lit/ds/symlink/ref3033.pdf" (at 59.69 140.97 0)
       (effects (font (size 1.27 1.27) italic) hide)
+    )
+    (property "MPN" "C2872391" (at 57.15 132.08 0)
+      (effects (font (size 1.27 1.27)) hide)
     )
     (pin "1")
@@
       (effects (font (size 1.27 1.27)) hide)
     )
+    (property "MPN" "C96446" (at 146.05 102.87 0)
+      (effects (font (size 1.27 1.27)) hide)
+    )
+    (property "Rating" "25V" (at 146.05 102.87 0)
+      (effects (font (size 1.27 1.27)) hide)
+    )
     (pin "1")
     (pin "2")
@@
       (effects (font (size 1.27 1.27)) hide)
     )
+    (property "MPN" "C1523" (at 166.37 34.29 0)
+      (effects (font (size 1.27 1.27)) hide)
+    )
+    (property "Rating" "50V" (at 166.37 34.29 0)
+      (effects (font (size 1.27 1.27)) hide)
+    )
     (pin "1")
     (pin "2")
@@
     (property "Rating" "63mW" (at 45.72 49.53 90)
       (effects (font (size 1.27 1.27)))
+    )
+    (property "MPN" "C11702" (at 45.72 46.99 0)
+      (effects (font (size 1.27 1.27)) hide)
     )
     (pin "1")
@@
       (effects (font (size 1.27 1.27)) (justify right))
     )
+    (property "MPN" "C174169" (at 81.28 40.64 0)
+      (effects (font (size 1.27 1.27)) hide)
+    )
     (pin "1")
     (pin "2")
@@
       (effects (font (size 1.27 1.27)) hide)
     )
+    (property "MPN" "C96446" (at 85.09 139.7 0)
+      (effects (font (size 1.27 1.27)) hide)
+    )
+    (property "Rating" "25V" (at 85.09 139.7 0)
+      (effects (font (size 1.27 1.27)) hide)
+    )
     (pin "1")
     (pin "2")
@@
       (effects (font (size 1.27 1.27)))
     )
-    (property "MPN" "" (at 36.83 121.92 0)
+    (property "MPN" "C17720" (at 36.83 121.92 0)
       (effects (font (size 1.27 1.27)) hide)
     )
@@
     )
     (property "Datasheet" "~" (at 63.5 53.34 0)
+      (effects (font (size 1.27 1.27)) hide)
+    )
+    (property "MPN" "C1527" (at 63.5 53.34 0)
+      (effects (font (size 1.27 1.27)) hide)
+    )
+    (property "Rating" "50V" (at 63.5 53.34 0)
       (effects (font (size 1.27 1.27)) hide)
     )
@@
       (effects (font (size 1.27 1.27)))
     )
+    (property "MPN" "C25768" (at 147.32 49.53 0)
+      (effects (font (size 1.27 1.27)) hide)
+    )
     (pin "1")
     (pin "2")
@@
       (effects (font (size 1.27 1.27)) hide)
     )
+    (property "MPN" "C96446" (at 85.09 102.87 0)
+      (effects (font (size 1.27 1.27)) hide)
+    )
+    (property "Rating" "25V" (at 85.09 102.87 0)
+      (effects (font (size 1.27 1.27)) hide)
+    )
     (pin "1")
     (pin "2")
@@
       (effects (font (size 1.27 1.27)) hide)
     )
-    (property "Datasheet" " ~" (at 26.67 46.99 0)
+    (property "Datasheet" "~" (at 26.67 46.99 0)
       (effects (font (size 1.27 1.27)) hide)
     )
@@
       (effects (font (size 1.27 1.27)))
     )
+    (property "MPN" "C11702" (at 217.17 52.07 0)
+      (effects (font (size 1.27 1.27)) hide)
+    )
     (pin "1")
     (pin "2")
@@
     (property "Rating" "63mW" (at 160.02 52.07 90)
       (effects (font (size 1.27 1.27)))
+    )
+    (property "MPN" "C25752" (at 160.02 49.53 0)
+      (effects (font (size 1.27 1.27)) hide)
     )
     (pin "1")
@@
       (effects (font (size 1.27 1.27)))
     )
+    (property "MPN" "C174169" (at 52.07 53.34 0)
+      (effects (font (size 1.27 1.27)) hide)
+    )
     (pin "1")
     (pin "2")
@@
       (effects (font (size 1.27 1.27)) (justify left))
     )
-    (property "Value" "MCP6001T-E/OT" (at 193.04 57.15 0)
+    (property "Value" "TLV9001IDBVR" (at 193.04 57.15 0)
       (effects (font (size 1.27 1.27)) (justify left))
     )
@@
       (effects (font (size 1.27 1.27)) (justify left) hide)
     )
-    (property "Datasheet" "http://ww1.microchip.com/downloads/en/DeviceDoc/21733j.pdf" (at 194.31 46.99 0)
+    (property "Datasheet" "https://www.ti.com/lit/ds/symlink/tlv9001.pdf?ts=1684276162908&ref_url=https%253A%252F%252Fwww.ti.com%252Fproduct%252FTLV9001" (at 194.31 46.99 0)
+      (effects (font (size 1.27 1.27)) hide)
+    )
+    (property "MPN" "C398363" (at 194.31 52.07 0)
       (effects (font (size 1.27 1.27)) hide)
     )
@@
       (effects (font (size 1.27 1.27)))
     )
+    (property "MPN" "C11702" (at 217.17 72.39 0)
+      (effects (font (size 1.27 1.27)) hide)
+    )
     (pin "1")
     (pin "2")
@@
       (effects (font (size 1.27 1.27)))
     )
+    (property "MPN" "C25917" (at 134.62 49.53 0)
+      (effects (font (size 1.27 1.27)) hide)
+    )
     (pin "1")
     (pin "2")
@@
       (effects (font (size 1.27 1.27)) hide)
     )
+    (property "MPN" "C1527" (at 223.52 62.23 0)
+      (effects (font (size 1.27 1.27)) hide)
+    )
+    (property "Rating" "50V" (at 223.52 62.23 0)
+      (effects (font (size 1.27 1.27)) hide)
+    )
     (pin "1")
     (pin "2")
@@
       (effects (font (size 1.27 1.27)) hide)
     )
+    (property "MPN" "C1523" (at 140.97 55.88 0)
+      (effects (font (size 1.27 1.27)) hide)
+    )
+    (property "Rating" "50V" (at 140.97 55.88 0)
+      (effects (font (size 1.27 1.27)) hide)
+    )

Commit message: Cleanup, minor bom changes and finished production files
Parts:
- D301: value PESD3V3L1BA,115 -> PESD3V3L1BA; MPN C51450 -> C2939000; Rating 5.8V 26V -> 4V 10.5V
Changed lines of the file:
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@@
       (effects (font (size 1.27 1.27)) (justify left))
     )
-    (property "Value" "PESD3V3L1BA,115" (at 30.48 60.96 90)
+    (property "Value" "PESD3V3L1BA" (at 30.48 60.96 90)
       (effects (font (size 1.27 1.27)) (justify left))
     )
@@
       (effects (font (size 1.27 1.27)) hide)
     )
-    (property "MPN" "C51450" (at 39.37 53.34 0)
+    (property "MPN" "C2939000" (at 39.37 53.34 0)
       (effects (font (size 1.27 1.27)) hide)
     )
-    (property "Rating" "5.8V 26V" (at 39.37 53.34 0)
+    (property "Rating" "4V 10.5V" (at 39.37 53.34 0)
       (effects (font (size 1.27 1.27)) hide)
     )
