File: hardware/dac.kicad_sch (KiCad schematic)
At the start: 17 parts, among them J401 031-5640-1010, U401 DAC7563SDGSR, U402 MCP6001T-E/OT

Commit message: Finished mcu schematic with the rp2040
Parts:
- U401: value DAC7563SDGSR -> DAC7562SDGSR; MPN DAC7563SDGSR -> C1554786
Changed lines of the file:
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@@
       (effects (font (size 1.27 1.27)) (justify right))
     )
-    (property "Value" "DAC7563SDGSR" (at 97.79 113.03 0)
+    (property "Value" "DAC7562SDGSR" (at 97.79 113.03 0)
       (effects (font (size 1.27 1.27)) (justify right))
     )
@@
       (effects (font (size 1.27 1.27)) hide)
     )
-    (property "Datasheet" "" (at 95.25 100.33 0)
+    (property "Datasheet" "https://www.ti.com/lit/ds/symlink/dac7562.pdf?ts=1683401788083&ref_url=https%253A%252F%252Fwww.ti.com%252Fproduct%252FDAC7562%252Fpart-details%252FDAC7562SDGSR" (at 95.25 100.33 0)
       (effects (font (size 1.27 1.27)) hide)
     )
@@
       (effects (font (size 1.27 1.27)))
     )
-    (property "MPN" "DAC7563SDGSR" (at 95.25 100.33 0)
+    (property "MPN" "C1554786" (at 95.25 100.33 0)
       (effects (font (size 1.27 1.27)) hide)
     )

Commit message: Finished routing
Parts:
- C402, C407: MPN CC0402KRX5R6BB104 -> C1525; Rating 10V -> 16V
Other:
- moved on the sheet: C404, C406
Changed lines of the file:
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@@
     (stroke (width 0) (type default))
   )
-  (wire (pts (xy 148.59 95.25) (xy 148.59 92.71))
+  (wire (pts (xy 148.59 99.06) (xy 148.59 92.71))
     (stroke (width 0) (type default))
   )
@@
     (stroke (width 0) (type default))
   )
-  (wire (pts (xy 173.99 102.87) (xy 173.99 105.41))
+  (wire (pts (xy 173.99 106.68) (xy 173.99 109.22))
     (stroke (width 0) (type default))
   )
@@
     (stroke (width 0) (type default))
   )
-  (wire (pts (xy 173.99 95.25) (xy 173.99 92.71))
+  (wire (pts (xy 173.99 99.06) (xy 173.99 92.71))
     (stroke (width 0) (type default))
   )
@@
     (stroke (width 0) (type default))
   )
-  (wire (pts (xy 148.59 102.87) (xy 148.59 105.41))
+  (wire (pts (xy 148.59 106.68) (xy 148.59 109.22))
     (stroke (width 0) (type default))
   )
@@
     )
   )
-  (symbol (lib_id "power:GND") (at 148.59 105.41 0) (unit 1)
-    (in_bom yes) (on_board yes) (dnp no)
-    (property "Reference" "#PWR0404" (at 148.59 111.76 0)
-      (effects (font (size 1.27 1.27)) hide)
-    )
-    (property "Value" "GND" (at 148.59 109.22 0)
-      (effects (font (size 1.27 1.27)) hide)
-    )
-    (property "Footprint" "" (at 148.59 105.41 0)
-      (effects (font (size 1.27 1.27)) hide)
-    )
-    (property "Datasheet" "" (at 148.59 105.41 0)
+  (symbol (lib_id "power:GND") (at 148.59 109.22 0) (unit 1)
+    (in_bom yes) (on_board yes) (dnp no)
+    (property "Reference" "#PWR0404" (at 148.59 115.57 0)
+      (effects (font (size 1.27 1.27)) hide)
+    )
+    (property "Value" "GND" (at 148.59 113.03 0)
+      (effects (font (size 1.27 1.27)) hide)
+    )
+    (property "Footprint" "" (at 148.59 109.22 0)
+      (effects (font (size 1.27 1.27)) hide)
+    )
+    (property "Datasheet" "" (at 148.59 109.22 0)
       (effects (font (size 1.27 1.27)) hide)
     )
@@
       (effects (font (size 1.27 1.27)) hide)
     )
-    (property "MPN" "CC0402KRX5R6BB104" (at 189.23 85.09 0)
-      (effects (font (size 1.27 1.27)) hide)
-    )
-    (property "Rating" "10V" (at 189.23 85.09 0)
+    (property "MPN" "C1525" (at 189.23 85.09 0)
+      (effects (font (size 1.27 1.27)) hide)
+    )
+    (property "Rating" "16V" (at 189.23 85.09 0)
       (effects (font (size 1.27 1.27)) hide)
     )
@@
     )
   )
-  (symbol (lib_id "Device:C") (at 173.99 99.06 0) (unit 1)
-    (in_bom yes) (on_board yes) (dnp no)
-    (property "Reference" "C406" (at 177.8 97.79 0)
-      (effects (font (size 1.27 1.27)) (justify left))
-    )
-    (property "Value" "150p" (at 177.8 100.33 0)
-      (effects (font (size 1.27 1.27)) (justify left))
-    )
-    (property "Footprint" "Capacitor_SMD:C_0402_1005Metric" (at 174.9552 102.87 0)
-      (effects (font (size 1.27 1.27)) hide)
-    )
-    (property "Datasheet" "~" (at 173.99 99.06 0)
+  (symbol (lib_id "Device:C") (at 173.99 102.87 0) (unit 1)
+    (in_bom yes) (on_board yes) (dnp no)
+    (property "Reference" "C406" (at 177.8 101.6 0)
+      (effects (font (size 1.27 1.27)) (justify left))
+    )
+    (property "Value" "150p" (at 177.8 104.14 0)
+      (effects (font (size 1.27 1.27)) (justify left))
+    )
+    (property "Footprint" "Capacitor_SMD:C_0402_1005Metric" (at 174.9552 106.68 0)
+      (effects (font (size 1.27 1.27)) hide)
+    )
+    (property "Datasheet" "~" (at 173.99 102.87 0)
       (effects (font (size 1.27 1.27)) hide)
     )
@@
     )
   )
-  (symbol (lib_id "Device:C") (at 148.59 99.06 0) (unit 1)
-    (in_bom yes) (on_board yes) (dnp no)
-    (property "Reference" "C404" (at 152.4 97.79 0)
-      (effects (font (size 1.27 1.27)) (justify left))
-    )
-    (property "Value" "1n" (at 152.4 100.33 0)
-      (effects (font (size 1.27 1.27)) (justify left))
-    )
-    (property "Footprint" "Capacitor_SMD:C_0402_1005Metric" (at 149.5552 102.87 0)
-      (effects (font (size 1.27 1.27)) hide)
-    )
-    (property "Datasheet" "~" (at 148.59 99.06 0)
+  (symbol (lib_id "Device:C") (at 148.59 102.87 0) (unit 1)
+    (in_bom yes) (on_board yes) (dnp no)
+    (property "Reference" "C404" (at 152.4 101.6 0)
+      (effects (font (size 1.27 1.27)) (justify left))
+    )
+    (property "Value" "1n" (at 152.4 104.14 0)
+      (effects (font (size 1.27 1.27)) (justify left))
+    )
+    (property "Footprint" "Capacitor_SMD:C_0402_1005Metric" (at 149.5552 106.68 0)
+      (effects (font (size 1.27 1.27)) hide)
+    )
+    (property "Datasheet" "~" (at 148.59 102.87 0)
       (effects (font (size 1.27 1.27)) hide)
     )
@@
     )
   )
-  (symbol (lib_id "power:GND") (at 173.99 105.41 0) (unit 1)
-    (in_bom yes) (on_board yes) (dnp no)
-    (property "Reference" "#PWR0405" (at 173.99 111.76 0)
-      (effects (font (size 1.27 1.27)) hide)
-    )
-    (property "Value" "GND" (at 173.99 109.22 0)
-      (effects (font (size 1.27 1.27)) hide)
-    )
-    (property "Footprint" "" (at 173.99 105.41 0)
-      (effects (font (size 1.27 1.27)) hide)
-    )
-    (property "Datasheet" "" (at 173.99 105.41 0)
+  (symbol (lib_id "power:GND") (at 173.99 109.22 0) (unit 1)
+    (in_bom yes) (on_board yes) (dnp no)
+    (property "Reference" "#PWR0405" (at 173.99 115.57 0)
+      (effects (font (size 1.27 1.27)) hide)
+    )
+    (property "Value" "GND" (at 173.99 113.03 0)
+      (effects (font (size 1.27 1.27)) hide)
+    )
+    (property "Footprint" "" (at 173.99 109.22 0)
+      (effects (font (size 1.27 1.27)) hide)
+    )
+    (property "Datasheet" "" (at 173.99 109.22 0)
       (effects (font (size 1.27 1.27)) hide)
     )
@@
       (effects (font (size 1.27 1.27)) hide)
     )
-    (property "MPN" "CC0402KRX5R6BB104" (at 82.55 77.47 0)
-      (effects (font (size 1.27 1.27)) hide)
-    )
-    (property "Rating" "10V" (at 82.55 77.47 0)
-      (effects (font (size 1.27 1.27)) hide)
-    )
+    (property "MPN" "C1525" (at 82.55 77.47 0)
+      (effects (font (size 1.27 1.27)) hide)
+    )
+    (property "Rating" "16V" (at 82.55 77.47 0)
+      (effects (font (size 1.27 1.27)) hide)
+    )

Commit message: Finished bom
Parts:
- C401: MPN (none) -> C96446; Rating (none) -> 25V
- C403: MPN CC0603KRX5R6BB105 -> C15849; Rating 10V -> 50V
- C404, C405: MPN (none) -> C1523; Rating (none) -> 50V
- C406: MPN (none) -> C1527; Rating (none) -> 50V
- D401: MPN (none) -> C51450; Rating (none) -> 5.8V 26V
- R401: MPN (none) -> C17168
- R402: MPN (none) -> C25744
- R403: MPN (none) -> C25917
- R404: MPN (none) -> C25768
- R405: MPN (none) -> C25752
- R406: MPN (none) -> C25120
- U402: value MCP6001T-E/OT -> TLV9001IDBVR; MPN (none) -> C398363
Changed lines of the file:
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@@
       (effects (font (size 1.27 1.27)))
+    )
+    (property "MPN" "C25917" (at 142.24 92.71 0)
+      (effects (font (size 1.27 1.27)) hide)
     )
     (pin "1")
@@
       (effects (font (size 1.27 1.27)) (justify left))
     )
+    (property "MPN" "C25744" (at 133.35 109.22 0)
+      (effects (font (size 1.27 1.27)) hide)
+    )
     (pin "1")
     (pin "2")
@@
       (effects (font (size 1.27 1.27)) hide)
     )
-    (property "Datasheet" " ~" (at 250.19 95.25 0)
+    (property "Datasheet" "~" (at 250.19 95.25 0)
       (effects (font (size 1.27 1.27)) hide)
     )
@@
       (effects (font (size 1.27 1.27)) (justify left))
     )
-    (property "Value" "MCP6001T-E/OT" (at 200.66 100.33 0)
+    (property "Value" "TLV9001IDBVR" (at 200.66 100.33 0)
       (effects (font (size 1.27 1.27)) (justify left))
     )
@@
       (effects (font (size 1.27 1.27)) (justify left) hide)
     )
-    (property "Datasheet" "http://ww1.microchip.com/downloads/en/DeviceDoc/21733j.pdf" (at 201.93 90.17 0)
+    (property "Datasheet" "https://www.ti.com/lit/ds/symlink/tlv9001.pdf?ts=1684276162908&ref_url=https%253A%252F%252Fwww.ti.com%252Fproduct%252FTLV9001" (at 201.93 90.17 0)
+      (effects (font (size 1.27 1.27)) hide)
+    )
+    (property "MPN" "C398363" (at 201.93 95.25 0)
       (effects (font (size 1.27 1.27)) hide)
     )
@@
       (effects (font (size 1.27 1.27)) hide)
     )
+    (property "MPN" "C96446" (at 69.85 77.47 0)
+      (effects (font (size 1.27 1.27)) hide)
+    )
+    (property "Rating" "25V" (at 69.85 77.47 0)
+      (effects (font (size 1.27 1.27)) hide)
+    )
     (pin "1")
     (pin "2")
@@
     )
     (property "Datasheet" "~" (at 173.99 102.87 0)
+      (effects (font (size 1.27 1.27)) hide)
+    )
+    (property "MPN" "C1527" (at 173.99 102.87 0)
+      (effects (font (size 1.27 1.27)) hide)
+    )
+    (property "Rating" "50V" (at 173.99 102.87 0)
       (effects (font (size 1.27 1.27)) hide)
     )
@@
       (effects (font (size 1.27 1.27)))
     )
+    (property "MPN" "C25120" (at 224.79 95.25 0)
+      (effects (font (size 1.27 1.27)) hide)
+    )
     (pin "1")
     (pin "2")
@@
       (effects (font (size 1.27 1.27)) hide)
     )
-    (property "MPN" "CC0603KRX5R6BB105" (at 120.65 109.22 0)
-      (effects (font (size 1.27 1.27)) hide)
-    )
-    (property "Rating" "10V" (at 120.65 109.22 0)
+    (property "MPN" "C15849" (at 120.65 109.22 0)
+      (effects (font (size 1.27 1.27)) hide)
+    )
+    (property "Rating" "50V" (at 120.65 109.22 0)
       (effects (font (size 1.27 1.27)) hide)
     )
@@
       (effects (font (size 1.27 1.27)))
     )
+    (property "MPN" "C25752" (at 167.64 92.71 0)
+      (effects (font (size 1.27 1.27)) hide)
+    )
     (pin "1")
     (pin "2")
@@
       (effects (font (size 1.27 1.27)) hide)
     )
+    (property "MPN" "C51450" (at 231.14 101.6 0)
+      (effects (font (size 1.27 1.27)) hide)
+    )
+    (property "Rating" "5.8V 26V" (at 231.14 101.6 0)
+      (effects (font (size 1.27 1.27)) hide)
+    )
     (pin "1")
     (pin "2")
@@
       (effects (font (size 1.27 1.27)) hide)
     )
+    (property "MPN" "C1523" (at 148.59 102.87 0)
+      (effects (font (size 1.27 1.27)) hide)
+    )
+    (property "Rating" "50V" (at 148.59 102.87 0)
+      (effects (font (size 1.27 1.27)) hide)
+    )
     (pin "1")
     (pin "2")
@@
       (effects (font (size 1.27 1.27)) hide)
     )
+    (property "MPN" "C1523" (at 173.99 77.47 0)
+      (effects (font (size 1.27 1.27)) hide)
+    )
+    (property "Rating" "50V" (at 173.99 77.47 0)
+      (effects (font (size 1.27 1.27)) hide)
+    )
     (pin "1")
     (pin "2")
@@
       (effects (font (size 1.27 1.27)))
     )
+    (property "MPN" "C25768" (at 154.94 92.71 0)
+      (effects (font (size 1.27 1.27)) hide)
+    )
     (pin "1")
     (pin "2")
@@
       (effects (font (size 1.27 1.27)))
     )
-    (pin "1")
+    (property "MPN" "C17168" (at 64.77 96.52 0)
+      (effects (font (size 1.27 1.27)) hide)
+    )
+    (pin "1")

Commit message: Cleanup, minor bom changes and finished production files
Parts:
- D401: value PESD3V3L1BA,115 -> PESD3V3L1BA; MPN C51450 -> C2939000; Rating 5.8V 26V -> 4V 10.5V
Changed lines of the file:
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@@
       (effects (font (size 1.27 1.27)) (justify left))
     )
-    (property "Value" "PESD3V3L1BA,115" (at 231.14 106.68 90)
+    (property "Value" "PESD3V3L1BA" (at 231.14 106.68 90)
       (effects (font (size 1.27 1.27)) (justify left))
     )
@@
       (effects (font (size 1.27 1.27)) hide)
     )
-    (property "MPN" "C51450" (at 231.14 101.6 0)
+    (property "MPN" "C2939000" (at 231.14 101.6 0)
       (effects (font (size 1.27 1.27)) hide)
     )
-    (property "Rating" "5.8V 26V" (at 231.14 101.6 0)
+    (property "Rating" "4V 10.5V" (at 231.14 101.6 0)
       (effects (font (size 1.27 1.27)) hide)
     )
