File: hardware/power.kicad_sch (KiCad schematic)
At the start: 27 parts, among them U101 TLV62569DBV, U102 HT7533-1, U103 MCP6001T-E/OT

Commit message: Finished routing
Parts:
- C101, C102: MPN CC0603KRX5R6BB105 -> C15849; Rating 10V -> 50V
- C103, C104, C106, C107, C108: MPN CC0805KRX5R6BB225 -> C45783; Rating 10V -> 25V
- C109: MPN CC0402KRX5R6BB104 -> C1525; Rating 10V -> 16V
- L101: MPN (none) -> C961338
- L102: MPN (none) -> C408441; Rating (none) -> 16A
- R101: MPN (none) -> C17415
Other:
- moved on the sheet: C105, D101, R102, R103, R104

Commit message: Finished bom
Parts:
- D101, D102: MPN (none) -> C2292
- R102: MPN (none) -> C321525
- R103: MPN (none) -> C25741
- R104, R105, R106, R107: MPN (none) -> C11702
- U101: MPN (none) -> C141836
- U102: MPN (none) -> C14289
- U103: value MCP6001T-E/OT -> TLV9001IDBVR; MPN (none) -> C398363
Changed lines of the file:
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@@
       (effects (font (size 1.27 1.27)) (justify left))
+    )
+    (property "MPN" "C321525" (at 115.57 116.84 0)
+      (effects (font (size 1.27 1.27)) hide)
     )
     (pin "1")
@@
       (effects (font (size 1.27 1.27)))
     )
+    (property "MPN" "C2292" (at 142.24 118.11 0)
+      (effects (font (size 1.27 1.27)) hide)
+    )
     (pin "1")
     (pin "2")
@@
       (effects (font (size 1.27 1.27)) (justify left))
     )
+    (property "MPN" "C11702" (at 179.07 71.12 0)
+      (effects (font (size 1.27 1.27)) hide)
+    )
     (pin "1")
     (pin "2")
@@
     (property "Rating" "63mW" (at 147.32 134.62 0)
       (effects (font (size 1.27 1.27)))
+    )
+    (property "MPN" "C11702" (at 142.24 130.81 0)
+      (effects (font (size 1.27 1.27)) hide)
     )
     (pin "1")
@@
     )
     (property "Datasheet" "http://www.ti.com/lit/ds/symlink/tlv62569.pdf" (at 67.31 100.33 0)
+      (effects (font (size 1.27 1.27)) hide)
+    )
+    (property "MPN" "C141836" (at 73.66 111.76 0)
       (effects (font (size 1.27 1.27)) hide)
     )
@@
       (effects (font (size 1.27 1.27)) hide)
     )
+    (property "MPN" "C14289" (at 121.92 58.42 0)
+      (effects (font (size 1.27 1.27)) hide)
+    )
     (pin "1")
     (pin "2")
@@
       (effects (font (size 1.27 1.27)))
     )
+    (property "MPN" "C2292" (at 149.86 62.23 0)
+      (effects (font (size 1.27 1.27)) hide)
+    )
     (pin "1")
     (pin "2")
@@
       (effects (font (size 1.27 1.27)) (justify left))
     )
+    (property "MPN" "C11702" (at 179.07 59.69 0)
+      (effects (font (size 1.27 1.27)) hide)
+    )
     (pin "1")
     (pin "2")
@@
       (effects (font (size 1.27 1.27)) (justify left))
     )
+    (property "MPN" "C25741" (at 115.57 132.08 0)
+      (effects (font (size 1.27 1.27)) hide)
+    )
     (pin "1")
     (pin "2")
@@
       (effects (font (size 1.27 1.27)))
     )
-    (property "Value" "MCP6001T-E/OT" (at 226.06 71.12 0)
+    (property "Value" "TLV9001IDBVR" (at 226.06 71.12 0)
       (effects (font (size 1.27 1.27)))
     )
@@
       (effects (font (size 1.27 1.27)) (justify left) hide)
     )
-    (property "Datasheet" "http://ww1.microchip.com/downloads/en/DeviceDoc/21733j.pdf" (at 218.44 62.23 0)
+    (property "Datasheet" "https://www.ti.com/lit/ds/symlink/tlv9001.pdf?ts=1684276162908&ref_url=https%253A%252F%252Fwww.ti.com%252Fproduct%252FTLV9001" (at 218.44 62.23 0)
+      (effects (font (size 1.27 1.27)) hide)
+    )
+    (property "MPN" "C398363" (at 218.44 67.31 0)
       (effects (font (size 1.27 1.27)) hide)
     )
@@
       (effects (font (size 1.27 1.27)) (justify left))
     )
-    (pin "1")
+    (property "MPN" "C11702" (at 149.86 72.39 0)
+      (effects (font (size 1.27 1.27)) hide)
+    )
+    (pin "1")

Commit message: Cleanup, minor bom changes and finished production files
Parts:
- D101, D102: MPN C2292 -> C72043
- L101: MPN C961338 -> C361500
Changed lines of the file:
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@@
       (effects (font (size 1.27 1.27)))
     )
-    (property "MPN" "C2292" (at 142.24 118.11 0)
+    (property "MPN" "C72043" (at 142.24 118.11 0)
       (effects (font (size 1.27 1.27)) hide)
     )
@@
       (effects (font (size 1.27 1.27)))
     )
-    (property "MPN" "C2292" (at 149.86 62.23 0)
+    (property "MPN" "C72043" (at 149.86 62.23 0)
       (effects (font (size 1.27 1.27)) hide)
     )
@@
       (effects (font (size 1.27 1.27)))
     )
-    (property "MPN" "C961338" (at 44.45 55.88 0)
-      (effects (font (size 1.27 1.27)) hide)
-    )
+    (property "MPN" "C361500" (at 44.45 55.88 0)
+      (effects (font (size 1.27 1.27)) hide)
+    )
