File: hardware/rp2040_audioboard.kicad_sch (KiCad schematic)
At the start: 4 parts

Commit message: Finished mcu schematic with the rp2040
Other:
- sheet [2] MCU ports: added ADC_SPI1_CLK, ADC_SPI1_MISO, ADC_SPI1_NCS, DAC_SPI0_CLK, DAC_SPI0_MOSI, DAC_SPI0_NCS; removed SPI1_MISO, SPI1_NSS, SPI1_SCK, SPI2_MOSI, SPI2_NSS, SPI2_SCK
Changed lines of the file:
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@@
+    (stroke (width 0) (type default))
+  )
+  (wire (pts (xy 81.28 118.11) (xy 99.06 118.11))
+    (stroke (width 0) (type default))
+  )
+  (wire (pts (xy 81.28 85.09) (xy 99.06 85.09))
+    (stroke (width 0) (type default))
+  )
+  (wire (pts (xy 266.7 146.05) (xy 266.7 149.86))
+    (stroke (width 0) (type default))
+  )
+  (polyline (pts (xy 224.79 127) (xy 224.79 161.29))
+    (stroke (width 0) (type default))
+  )
+  (wire (pts (xy 246.38 149.86) (xy 251.46 149.86))
+    (stroke (width 0) (type default))
+  )
+  (polyline (pts (xy 278.13 161.29) (xy 278.13 127))
+    (stroke (width 0) (type default))
+  )
+  (wire (pts (xy 81.28 87.63) (xy 99.06 87.63))
+    (stroke (width 0) (type default))
+  )
+  (wire (pts (xy 81.28 125.73) (xy 99.06 125.73))
+    (stroke (width 0) (type default))
+  )
+  (wire (pts (xy 256.54 149.86) (xy 266.7 149.86))
+    (stroke (width 0) (type default))
+  )
+  (wire (pts (xy 237.49 149.86) (xy 246.38 149.86))
+    (stroke (width 0) (type default))
+  )
+  (wire (pts (xy 256.54 146.05) (xy 256.54 149.86))
+    (stroke (width 0) (type default))
+  )
+  (polyline (pts (xy 224.79 161.29) (xy 278.13 161.29))
+    (stroke (width 0) (type default))
+  )
+  (wire (pts (xy 81.28 90.17) (xy 99.06 90.17))
+    (stroke (width 0) (type default))
+  )
+  (wire (pts (xy 237.49 146.05) (xy 237.49 149.86))
+    (stroke (width 0) (type default))
+  )
+  (wire (pts (xy 81.28 123.19) (xy 99.06 123.19))
+    (stroke (width 0) (type default))
+  )
+  (wire (pts (xy 81.28 128.27) (xy 99.06 128.27))
+    (stroke (width 0) (type default))
+  )
+  (polyline (pts (xy 224.79 127) (xy 278.13 127))
+    (stroke (width 0) (type default))
+  )
+  (wire (pts (xy 251.46 149.86) (xy 251.46 151.13))
+    (stroke (width 0) (type default))
+  )
+  (polyline (pts (xy 224.79 132.08) (xy 224.79 132.08))
     (stroke (width 0) (type default))
   )
   (wire (pts (xy 81.28 120.65) (xy 99.06 120.65))
-    (stroke (width 0) (type default))
-  )
-  (wire (pts (xy 81.28 85.09) (xy 99.06 85.09))
-    (stroke (width 0) (type default))
-  )
-  (wire (pts (xy 266.7 146.05) (xy 266.7 149.86))
-    (stroke (width 0) (type default))
-  )
-  (polyline (pts (xy 224.79 127) (xy 224.79 161.29))
-    (stroke (width 0) (type default))
-  )
-  (wire (pts (xy 246.38 149.86) (xy 251.46 149.86))
-    (stroke (width 0) (type default))
-  )
-  (polyline (pts (xy 278.13 161.29) (xy 278.13 127))
-    (stroke (width 0) (type default))
-  )
-  (wire (pts (xy 81.28 87.63) (xy 99.06 87.63))
-    (stroke (width 0) (type default))
-  )
-  (wire (pts (xy 81.28 125.73) (xy 99.06 125.73))
-    (stroke (width 0) (type default))
-  )
-  (wire (pts (xy 256.54 149.86) (xy 266.7 149.86))
-    (stroke (width 0) (type default))
-  )
-  (wire (pts (xy 81.28 118.11) (xy 99.06 118.11))
-    (stroke (width 0) (type default))
-  )
-  (wire (pts (xy 237.49 149.86) (xy 246.38 149.86))
-    (stroke (width 0) (type default))
-  )
-  (wire (pts (xy 256.54 146.05) (xy 256.54 149.86))
-    (stroke (width 0) (type default))
-  )
-  (polyline (pts (xy 224.79 161.29) (xy 278.13 161.29))
-    (stroke (width 0) (type default))
-  )
-  (wire (pts (xy 81.28 90.17) (xy 99.06 90.17))
-    (stroke (width 0) (type default))
-  )
-  (wire (pts (xy 237.49 146.05) (xy 237.49 149.86))
-    (stroke (width 0) (type default))
-  )
-  (wire (pts (xy 81.28 123.19) (xy 99.06 123.19))
-    (stroke (width 0) (type default))
-  )
-  (wire (pts (xy 81.28 128.27) (xy 99.06 128.27))
-    (stroke (width 0) (type default))
-  )
-  (polyline (pts (xy 224.79 127) (xy 278.13 127))
-    (stroke (width 0) (type default))
-  )
-  (wire (pts (xy 251.46 149.86) (xy 251.46 151.13))
-    (stroke (width 0) (type default))
-  )
-  (polyline (pts (xy 224.79 132.08) (xy 224.79 132.08))
     (stroke (width 0) (type default))
   )
@@
       (effects (font (size 1.27 1.27)) (justify right))
     )
-    (pin "SPI_CLK" input (at 81.28 120.65 0)
+    (pin "SPI_CLK" input (at 81.28 118.11 0)
       (effects (font (size 1.27 1.27)) (justify right))
     )
@@
       (effects (font (size 1.27 1.27)) (justify right))
     )
-    (pin "SPI_MOSI" input (at 81.28 118.11 0)
+    (pin "SPI_MOSI" input (at 81.28 120.65 0)
       (effects (font (size 1.27 1.27)) (justify right))
     )
@@
       (effects (font (size 1.27 1.27)) (justify left top))
     )
-    (pin "SPI1_NSS" output (at 99.06 87.63 180)
-      (effects (font (size 1.27 1.27)) (justify left))
-    )
-    (pin "SPI1_MISO" input (at 99.06 90.17 180)
-      (effects (font (size 1.27 1.27)) (justify left))
-    )
-    (pin "SPI2_MOSI" output (at 99.06 118.11 180)
-      (effects (font (size 1.27 1.27)) (justify left))
-    )
-    (pin "SPI2_NSS" output (at 99.06 123.19 180)
-      (effects (font (size 1.27 1.27)) (justify left))
-    )
     (pin "DAC_NLDAC" output (at 99.06 125.73 180)
       (effects (font (size 1.27 1.27)) (justify left))
@@
       (effects (font (size 1.27 1.27)) (justify left))
     )
-    (pin "SPI1_SCK" output (at 99.06 85.09 180)
-      (effects (font (size 1.27 1.27)) (justify left))
-    )
-    (pin "SPI2_SCK" output (at 99.06 120.65 180)
-      (effects (font (size 1.27 1.27)) (justify left))
-    )
+    (pin "ADC_SPI1_NCS" output (at 99.06 87.63 180)
+      (effects (font (size 1.27 1.27)) (justify left))
+    )
+    (pin "ADC_SPI1_MISO" input (at 99.06 90.17 180)
+      (effects (font (size 1.27 1.27)) (justify left))
+    )
+    (pin "ADC_SPI1_CLK" output (at 99.06 85.09 180)
+      (effects (font (size 1.27 1.27)) (justify left))
+    )
+    (pin "DAC_SPI0_NCS" output (at 99.06 123.19 180)
+      (effects (font (size 1.27 1.27)) (justify left))
+    )
+    (pin "DAC_SPI0_MOSI" output (at 99.06 120.65 180)
+      (effects (font (size 1.27 1.27)) (justify left))
+    )
+    (pin "DAC_SPI0_CLK" output (at 99.06 118.11 180)
+      (effects (font (size 1.27 1.27)) (justify left))
+    )
